File: EATremoloSMD/EATremoloSMD.sch (KiCad schematic (older format))
At the start: 40 parts, among them J1 JACK__MONO_2P_NC, J2 BARREL_JACK, J3 JACK__MONO_2P_NC, Q1 Q_NJFET_DSG, Q2 Q_NPN_EBC, Q3 Q_NPN_EBC, Q4 Q_NJFET_DSG, SW1 SW_3PDT_on_on

Commit message: BoardUpdate
Parts:
- C1, C2, C3, C4, C5, C6, C7, C8, C9: footprint Capacitors_SMD:C_0402_NoSilk -> Capacitors_SMD:C_0805
- R1, R10, R11, R12, R13, R14, R15, R16, R2, R3, R4, R5, R6, R7, R8, R9: footprint Resistors_SMD:R_0402_NoSilk -> Resistors_SMD:R_0805
Changed lines of the file:
@@
 encoding utf-8
 Sheet 1 1
-Title ""
+Title "EA Tremolo"
 Date ""
-Rev ""
+Rev "R2"
 Comp ""
 Comment1 ""
 Comment2 ""
-Comment3 ""
-Comment4 ""
+Comment3 "8-pin connector to sister board for control pots/led indicator"
+Comment4 "Simple JFET controlled Tremolo "
 $EndDescr
 $Comp
@@
 F 0 "R1" H 3850 2050 50  0000 C CNN
 F 1 "1M" H 3850 2150 50  0000 C CNN
-F 2 "Resistors_SMD:R_0402_NoSilk" V 3630 2100 50  0001 C CNN
+F 2 "Resistors_SMD:R_0805" V 3630 2100 50  0001 C CNN
 F 3 "" H 3700 2100 50  0001 C CNN
 	1    3700 2100
@@
 F 0 "R3" H 4350 3400 50  0000 C CNN
 F 1 "1M" H 4350 3500 50  0000 C CNN
-F 2 "Resistors_SMD:R_0402_NoSilk" V 4130 3450 50  0001 C CNN
+F 2 "Resistors_SMD:R_0805" V 4130 3450 50  0001 C CNN
 F 3 "" H 4200 3450 50  0001 C CNN
 	1    4200 3450
@@
 F 0 "C1" V 3850 2950 50  0000 L CNN
 F 1 "47nF" V 4150 2950 50  0000 L CNN
-F 2 "Capacitors_SMD:C_0402_NoSilk" H 4038 2850 50  0001 C CNN
+F 2 "Capacitors_SMD:C_0805" H 4038 2850 50  0001 C CNN
 F 3 "" H 4000 3000 50  0001 C CNN
 	1    4000 3000
@@
 F 0 "R2" H 4350 2350 50  0000 C CNN
 F 1 "1M" H 4350 2450 50  0000 C CNN
-F 2 "Resistors_SMD:R_0402_NoSilk" V 4130 2400 50  0001 C CNN
+F 2 "Resistors_SMD:R_0805" V 4130 2400 50  0001 C CNN
 F 3 "" H 4200 2400 50  0001 C CNN
 	1    4200 2400
@@
 F 0 "R5" H 4550 3500 50  0000 C CNN
 F 1 "10K" H 4550 3400 50  0000 C CNN
-F 2 "Resistors_SMD:R_0402_NoSilk" V 4630 3450 50  0001 C CNN
+F 2 "Resistors_SMD:R_0805" V 4630 3450 50  0001 C CNN
 F 3 "" H 4700 3450 50  0001 C CNN
 	1    4700 3450
@@
 F 0 "C5" V 5300 2700 50  0000 L CNN
 F 1 "10uF" V 5000 2650 50  0000 L CNN
-F 2 "Capacitors_SMD:C_0402_NoSilk" H 5188 2550 50  0001 C CNN
+F 2 "Capacitors_SMD:C_0805" H 5188 2550 50  0001 C CNN
 F 3 "" H 5150 2700 50  0001 C CNN
 	1    5150 2700
@@
 F 0 "C6" V 5400 2650 50  0000 L CNN
 F 1 "220nF" V 5700 2600 50  0000 L CNN
-F 2 "Capacitors_SMD:C_0402_NoSilk" H 5588 2550 50  0001 C CNN
+F 2 "Capacitors_SMD:C_0805" H 5588 2550 50  0001 C CNN
 F 3 "" H 5550 2700 50  0001 C CNN
 	1    5550 2700
@@
 F 0 "R8" H 5650 3500 50  0000 C CNN
 F 1 "150K" H 5650 3400 50  0000 C CNN
-F 2 "Resistors_SMD:R_0402_NoSilk" V 5730 3450 50  0001 C CNN
+F 2 "Resistors_SMD:R_0805" V 5730 3450 50  0001 C CNN
 F 3 "" H 5800 3450 50  0001 C CNN
 	1    5800 3450
@@
 F 0 "R10" V 6280 2150 50  0000 C CNN
 F 1 "4.7K" V 6200 2150 50  0000 C CNN
-F 2 "Resistors_SMD:R_0402_NoSilk" V 6130 2150 50  0001 C CNN
+F 2 "Resistors_SMD:R_0805" V 6130 2150 50  0001 C CNN
 F 3 "" H 6200 2150 50  0001 C CNN
 	1    6200 2150
@@
 F 0 "R7" V 5880 2250 50  0000 C CNN
 F 1 "560K" V 5800 2250 50  0000 C CNN
-F 2 "Resistors_SMD:R_0402_NoSilk" V 5730 2250 50  0001 C CNN
+F 2 "Resistors_SMD:R_0805" V 5730 2250 50  0001 C CNN
 F 3 "" H 5800 2250 50  0001 C CNN
 	1    5800 2250
@@
 F 0 "R11" V 6350 3000 50  0000 C CNN
 F 1 "180R" V 6550 3000 50  0000 C CNN
-F 2 "Resistors_SMD:R_0402_NoSilk" V 6380 3000 50  0001 C CNN
+F 2 "Resistors_SMD:R_0805" V 6380 3000 50  0001 C CNN
 F 3 "" H 6450 3000 50  0001 C CNN
 	1    6450 3000
@@
 F 0 "R12" H 6850 3400 50  0000 C CNN
 F 1 "1.2K" H 6850 3500 50  0000 C CNN
-F 2 "Resistors_SMD:R_0402_NoSilk" V 6630 3450 50  0001 C CNN
+F 2 "Resistors_SMD:R_0805" V 6630 3450 50  0001 C CNN
 F 3 "" H 6700 3450 50  0001 C CNN
 	1    6700 3450
@@
 F 0 "C9" V 7100 3000 50  0000 L CNN
 F 1 "10uF" V 6800 3000 50  0000 L CNN
-F 2 "Capacitors_SMD:C_0402_NoSilk" H 6988 2850 50  0001 C CNN
+F 2 "Capacitors_SMD:C_0805" H 6988 2850 50  0001 C CNN
 F 3 "" H 6950 3000 50  0001 C CNN
 	1    6950 3000
@@
 F 0 "C7" V 6400 2350 50  0000 L CNN
 F 1 "470nF" V 6700 2350 50  0000 L CNN
-F 2 "Capacitors_SMD:C_0402_NoSilk" H 6588 2250 50  0001 C CNN
+F 2 "Capacitors_SMD:C_0805" H 6588 2250 50  0001 C CNN
 F 3 "" H 6550 2400 50  0001 C CNN
 	1    6550 2400
@@
 F 0 "R13" V 7080 4700 50  0000 C CNN
 F 1 "68k" V 7000 4700 50  0000 C CNN
-F 2 "Resistors_SMD:R_0402_NoSilk" V 6930 4700 50  0001 C CNN
+F 2 "Resistors_SMD:R_0805" V 6930 4700 50  0001 C CNN
 F 3 "" H 7000 4700 50  0001 C CNN
 	1    7000 4700
@@
 F 0 "C8" V 6050 5300 50  0000 L CNN
 F 1 "470nF" V 6350 5250 50  0000 L CNN
-F 2 "Capacitors_SMD:C_0402_NoSilk" H 6238 5200 50  0001 C CNN
+F 2 "Capacitors_SMD:C_0805" H 6238 5200 50  0001 C CNN
 F 3 "" H 6200 5350 50  0001 C CNN
 	1    6200 5350
@@
 F 0 "R6" V 5680 5350 50  0000 C CNN
 F 1 "2.2M" V 5600 5350 50  0000 C CNN
-F 2 "Resistors_SMD:R_0402_NoSilk" V 5530 5350 50  0001 C CNN
+F 2 "Resistors_SMD:R_0805" V 5530 5350 50  0001 C CNN
 F 3 "" H 5600 5350 50  0001 C CNN
 	1    5600 5350
@@
 F 0 "R9" H 10500 4950 50  0000 C CNN
 F 1 "10K" H 10500 5050 50  0000 C CNN
-F 2 "Resistors_SMD:R_0402_NoSilk" V 10280 5000 50  0001 C CNN
+F 2 "Resistors_SMD:R_0805" V 10280 5000 50  0001 C CNN
 F 3 "" H 10350 5000 50  0001 C CNN
 	1    10350 5000
@@
 F 0 "C3" V 4750 5650 50  0000 L CNN
 F 1 "1uF" V 4850 5650 50  0000 L CNN
-F 2 "Capacitors_SMD:C_0402_NoSilk" H 5038 5550 50  0001 C CNN
+F 2 "Capacitors_SMD:C_0805" H 5038 5550 50  0001 C CNN
 F 3 "" H 5000 5700 50  0001 C CNN
 	1    5000 5700
@@
 F 0 "C4" V 4850 6050 50  0000 L CNN
 F 1 "1uF" V 4750 6050 50  0000 L CNN
-F 2 "Capacitors_SMD:C_0402_NoSilk" H 5038 5950 50  0001 C CNN
+F 2 "Capacitors_SMD:C_0805" H 5038 5950 50  0001 C CNN
 F 3 "" H 5000 6100 50  0001 C CNN
 	1    5000 6100
@@
 F 0 "C2" H 4575 6000 50  0000 L CNN
 F 1 "1uF" H 4575 5800 50  0000 L CNN
-F 2 "Capacitors_SMD:C_0402_NoSilk" H 4588 5750 50  0001 C CNN
+F 2 "Capacitors_SMD:C_0805" H 4588 5750 50  0001 C CNN
 F 3 "" H 4550 5900 50  0001 C CNN
 	1    4550 5900
@@
 F 0 "R4" H 4700 6300 50  0000 C CNN
 F 1 "15K" H 4700 6400 50  0000 C CNN
-F 2 "Resistors_SMD:R_0402_NoSilk" V 4480 6350 50  0001 C CNN
+F 2 "Resistors_SMD:R_0805" V 4480 6350 50  0001 C CNN
 F 3 "" H 4550 6350 50  0001 C CNN
 	1    4550 6350
@@
 F 0 "R15" V 7080 4300 50  0000 C CNN
 F 1 "100K" V 7000 4300 50  0000 C CNN
-F 2 "Resistors_SMD:R_0402_NoSilk" V 6930 4300 50  0001 C CNN
+F 2 "Resistors_SMD:R_0805" V 6930 4300 50  0001 C CNN
 F 3 "" H 7000 4300 50  0001 C CNN
 	1    7000 4300
@@
 F 0 "R14" V 6780 4300 50  0000 C CNN
 F 1 "180K" V 6700 4300 50  0000 C CNN
-F 2 "Resistors_SMD:R_0402_NoSilk" V 6630 4300 50  0001 C CNN
+F 2 "Resistors_SMD:R_0805" V 6630 4300 50  0001 C CNN
 F 3 "" H 6700 4300 50  0001 C CNN
 	1    6700 4300
@@
 F 0 "R16" V 4330 5700 50  0000 C CNN
 F 1 "1K" V 4250 5700 50  0000 C CNN
-F 2 "Resistors_SMD:R_0402_NoSilk" V 4180 5700 50  0001 C CNN
+F 2 "Resistors_SMD:R_0805" V 4180 5700 50  0001 C CNN
 F 3 "" H 4250 5700 50  0001 C CNN
 	1    4250 5700

Commit message: Update
Parts:
- removed J_AUXTOMAIN1, J_MAINTOAUX1: CONN_01X08, Pin_Headers:Pin_Header_Straight_1x08_Pitch2.54mm, symbol CONN_01X08
- added J_AUX2MAIN_1, J_AUX2MAIN_2, J_MAIN2AUX_1, J_MAIN2AUX_2: CONN_01X04, Pin_Headers:Pin_Header_Straight_1x04_Pitch2.54mm, symbol CONN_01X04
- Q2, Q3: symbol Q_NPN_EBC -> Q_NPN_BEC
- R16: value 1K -> 4K7
Connections:
- net GND: now also Q2.2 (E), J_MAIN2AUX_1.3 (P3), J_MAIN2AUX_2.1 (P1); no longer Q2.1 (E)
- net LED_AN: now also SW1.3 (C), J_MAIN2AUX_2.4 (P4); no longer C3.1, C8.2, Q2.3 (C), R6.2
- net LED_CA: now also C3.1, C8.2, Q2.3 (C), R6.2, J_MAIN2AUX_1.4 (P4); no longer SW1.3 (C)
- net RATE_P1: now also J_MAIN2AUX_1.1 (P1), J_MAIN2AUX_1.2 (P2)
- net VOL_P2: now also J_MAIN2AUX_2.2 (P2)
- net VOL_P3: now also J_MAIN2AUX_2.3 (P3)
- net at Q3.1 (B): now also C6.1, R7.2, R8.1; no longer R11.2
- net at C4.2, R6.1: now also Q2.1 (B); no longer Q2.2 (B)
- net at VOL1.1: now also J_AUX2MAIN_2.3 (P3)
- net at VOL1.2: now also J_AUX2MAIN_2.2 (P2)
- net at VOL1.3: now also J_AUX2MAIN_2.1 (P1)
- net at R9.2: now also J_AUX2MAIN_2.4 (P4)
- net at RATE1.1: now also J_AUX2MAIN_1.3 (P3)
- net at RATE1.2: now also J_AUX2MAIN_1.2 (P2)
- net at RATE1.3: now also J_AUX2MAIN_1.1 (P1)
- net at DRATE1.1 (K): now also J_AUX2MAIN_1.4 (P4)
- new net: Q3.2 (E), R11.2
Other:
- moved on the sheet: DRATE1, R9, RATE1, VOL1
Changed lines of the file:
@@
 $EndDescr
 $Comp
-L Q_NPN_EBC Q3
+L Q_NPN_BEC Q3
 U 1 1 5A21A919
 P 6100 2700
@@
 $EndComp
 $Comp
-L Q_NPN_EBC Q2
+L Q_NPN_BEC Q2
 U 1 1 5A21A985
 P 5750 6100
@@
 L POT VOL1
 U 1 1 5A21F62F
-P 9800 4800
-F 0 "VOL1" V 9625 4800 50  0000 C CNN
-F 1 "A25K" V 9700 4800 50  0000 C CNN
-F 2 "Potentiometers:Potentiometer_Bourns_PTV09A-1_Horizontal" H 9800 4800 50  0001 C CNN
-F 3 "" H 9800 4800 50  0001 C CNN
-	1    9800 4800
-	0    1    1    0
+P 9850 5000
+F 0 "VOL1" V 9675 5000 50  0000 C CNN
+F 1 "A25K" V 9750 5000 50  0000 C CNN
+F 2 "Potentiometers:Potentiometer_Bourns_PTV09A-1_Horizontal" H 9850 5000 50  0001 C CNN
+F 3 "" H 9850 5000 50  0001 C CNN
+	1    9850 5000
+	1    0    0    -1
 $EndComp
 Text Label 8900 2600 0    60   ~ 0
@@
 L R R9
 U 1 1 5A220FAF
-P 10350 5000
-F 0 "R9" H 10500 4950 50  0000 C CNN
-F 1 "10K" H 10500 5050 50  0000 C CNN
-F 2 "Resistors_SMD:R_0805" V 10280 5000 50  0001 C CNN
-F 3 "" H 10350 5000 50  0001 C CNN
-	1    10350 5000
-	1    0    0    -1
+P 9950 4650
+F 0 "R9" H 10100 4600 50  0000 C CNN
+F 1 "10K" H 10100 4700 50  0000 C CNN
+F 2 "Resistors_SMD:R_0805" V 9880 4650 50  0001 C CNN
+F 3 "" H 9950 4650 50  0001 C CNN
+	1    9950 4650
+	0    -1   -1   0
 $EndComp
 Text Label 5850 6650 0    60   ~ 0
@@
 L POT RATE1
 U 1 1 5A224067
-P 9500 5050
-F 0 "RATE1" V 9325 5050 50  0000 C CNN
-F 1 "B100K" V 9400 5050 50  0000 C CNN
-F 2 "Potentiometers:Potentiometer_Bourns_PTV09A-1_Horizontal" H 9500 5050 50  0001 C CNN
-F 3 "" H 9500 5050 50  0001 C CNN
-	1    9500 5050
-	0    1    1    0
+P 9100 5000
+F 0 "RATE1" V 8925 5000 50  0000 C CNN
+F 1 "B100K" V 9000 5000 50  0000 C CNN
+F 2 "Potentiometers:Potentiometer_Bourns_PTV09A-1_Horizontal" H 9100 5000 50  0001 C CNN
+F 3 "" H 9100 5000 50  0001 C CNN
+	1    9100 5000
+	1    0    0    -1
 $EndComp
 Text Label 3550 6650 1    60   ~ 0
@@
 L LED DRATE1
 U 1 1 5A2316FC
-P 10100 4950
-F 0 "DRATE1" H 10100 5050 50  0000 C CNN
-F 1 "LED" H 10100 4850 50  0000 C CNN
-F 2 "LEDs:LED_D5.0mm" H 10100 4950 50  0001 C CNN
-F 3 "" H 10100 4950 50  0001 C CNN
-	1    10100 4950
-	0    -1   -1   0
+P 9600 4650
+F 0 "DRATE1" H 9600 4750 50  0000 C CNN
+F 1 "LED" H 9600 4550 50  0000 C CNN
+F 2 "LEDs:LED_D5.0mm" H 9600 4650 50  0001 C CNN
+F 3 "" H 9600 4650 50  0001 C CNN
+	1    9600 4650
+	1    0    0    -1
 $EndComp
 NoConn ~ 2150 5600
@@
 P 4250 5700
 F 0 "R16" V 4330 5700 50  0000 C CNN
-F 1 "1K" V 4250 5700 50  0000 C CNN
+F 1 "4K7" V 4250 5700 50  0000 C CNN
 F 2 "Resistors_SMD:R_0805" V 4180 5700 50  0001 C CNN
 F 3 "" H 4250 5700 50  0001 C CNN
@@
 Wire Wire Line
 	2150 5500 2500 5500
-Text Label 7900 5300 1    60   ~ 0
+Text Label 7600 5300 1    60   ~ 0
 RATE_P1
-Text Label 8000 5300 1    60   ~ 0
+Text Label 7700 5300 1    60   ~ 0
 RATE_P2
-Text Label 8100 5300 1    60   ~ 0
+Text Label 7800 5300 1    60   ~ 0
 RATE_P3
 Text Label 4050 5300 3    60   ~ 0
@@
 Text Label 3550 5300 3    60   ~ 0
 RATE_P3
-Text Label 8200 5300 1    60   ~ 0
+Text Label 8300 5300 1    60   ~ 0
 VOL_P1
-Text Label 8300 5300 1    60   ~ 0
+Text Label 8400 5300 1    60   ~ 0
 VOL_P2
-Text Label 8400 5300 1    60   ~ 0
+Text Label 8500 5300 1    60   ~ 0
 VOL_P3
 Text Label 8500 2400 0    60   ~ 0
@@
 Text Label 8050 2400 2    60   ~ 0
 VOL_P3
+Text Label 3950 4300 2    60   ~ 0
+LED_AN
+Text Label 8600 5300 1    60   ~ 0
+LED_AN
 Text Label 4650 4300 0    60   ~ 0
-LED_AN
-Text Label 8500 5300 1    60   ~ 0
-LED_AN
-Text Label 3950 4300 2    60   ~ 0
 LED_CA
-Text Label 8600 5300 1    60   ~ 0
+Text Label 7900 5300 1    60   ~ 0
 LED_CA
-$Comp
-L CONN_01X08 J_MAINTOAUX1
-U 1 1 5A310401
-P 8250 5650
-F 0 "J_MAINTOAUX1" H 8250 6100 50  0000 C CNN
-F 1 "CONN_01X08" V 8350 5650 50  0000 C CNN
-F 2 "Pin_Headers:Pin_Header_Straight_1x08_Pitch2.54mm" H 8250 5650 50  0001 C CNN
-F 3 "" H 8250 5650 50  0001 C CNN
-	1    8250 5650
-	0    1    1    0
-$EndComp
-$Comp
-L CONN_01X08 J_AUXTOMAIN1
-U 1 1 5A31068B
-P 9750 5650
-F 0 "J_AUXTOMAIN1" H 9750 6100 50  0000 C CNN
-F 1 "CONN_01X08" V 9850 5650 50  0000 C CNN
-F 2 "Pin_Headers:Pin_Header_Straight_1x08_Pitch2.54mm" H 9750 5650 50  0001 C CNN
-F 3 "" H 9750 5650 50  0001 C CNN
-	1    9750 5650
-	0    1    1    0
-$EndComp
-Wire Wire Line
-	7900 5300 7900 5450
-Wire Wire Line
-	8000 5300 8000 5450
-Wire Wire Line
-	8100 5300 8100 5450
-Wire Wire Line
-	8200 5300 8200 5450
+Wire Wire Line
+	7600 5300 7600 5450
+Wire Wire Line
+	7700 5300 7700 5450
+Wire Wire Line
+	7800 5300 7800 5450
 Wire Wire Line
 	8300 5300 8300 5450
@@
 	8500 5300 8500 5450
 Wire Wire Line
-	8600 5450 8600 5300
-Wire Wire Line
-	9350 5050 9350 5450
-Wire Wire Line
-	9350 5450 9400 5450
-Wire Wire Line
-	9500 5200 9500 5450
-Wire Wire Line
-	9650 5050 9650 5150
-Wire Wire Line
-	9650 5150 9600 5150
-Wire Wire Line
-	9600 5150 9600 5450
-Wire Wire Line
-	9650 4800 9650 5000
-Wire Wire Line
-	9650 5000 9700 5000
-Wire Wire Line
-	9700 5000 9700 5450
-Wire Wire Line
-	9800 4950 9800 5450
-Wire Wire Line
-	9950 4800 9950 5000
-Wire Wire Line
-	9950 5000 9900 5000
-Wire Wire Line
-	9900 5000 9900 5450
-Wire Wire Line
-	10000 5450 10000 5250
-Wire Wire Line
-	10000 5250 10100 5250
-Wire Wire Line
-	10100 5250 10100 5100
-Wire Wire Line
-	10100 4800 10100 4700
-Wire Wire Line
-	10100 4700 10350 4700
-Wire Wire Line
-	10350 4700 10350 4850
-Wire Wire Line
-	10350 5150 10350 5300
-Wire Wire Line
-	10350 5300 10100 5300
-Wire Wire Line
-	10100 5300 10100 5450
+	8600 5300 8600 5450
+Wire Wire Line
+	7900 5450 7900 5300
+Wire Wire Line
+	9100 5150 9100 5450
+Wire Wire Line
+	9200 5150 9200 5450
+Wire Wire Line
+	9300 4800 9300 5450
+Wire Wire Line
+	9850 5150 9850 5450
+Wire Wire Line
+	9950 5150 9950 5450
+Wire Wire Line
+	10050 4800 10050 5450
+Wire Wire Line
+	9400 4650 9400 5450
+Wire Wire Line
+	10150 4650 10150 5450
+$Comp
+L CONN_01X04 J_MAIN2AUX_1
+U 1 1 5A403A0C
+P 7750 5650
+F 0 "J_MAIN2AUX_1" V 7850 5650 50  0000 C CNN
+F 1 "CONN_01X04" V 7850 5650 50  0001 C CNN
+F 2 "Pin_Headers:Pin_Header_Straight_1x04_Pitch2.54mm" H 7750 5650 50  0001 C CNN
+F 3 "" H 7750 5650 50  0001 C CNN
+	1    7750 5650
+	0    -1   1    0
+$EndComp
+$Comp
+L CONN_01X04 J_MAIN2AUX_2
+U 1 1 5A403F4A
+P 8450 5650
+F 0 "J_MAIN2AUX_2" V 8550 5650 50  0000 C CNN
+F 1 "CONN_01X04" V 8550 5650 50  0001 C CNN
+F 2 "Pin_Headers:Pin_Header_Straight_1x04_Pitch2.54mm" H 8450 5650 50  0001 C CNN
+F 3 "" H 8450 5650 50  0001 C CNN
+	1    8450 5650
+	0    -1   1    0
+$EndComp
+$Comp
+L CONN_01X04 J_AUX2MAIN_1
+U 1 1 5A4049A0
+P 9250 5650
+F 0 "J_AUX2MAIN_1" V 9350 5650 50  0000 C CNN
+F 1 "CONN_01X04" V 9350 5650 50  0001 C CNN
+F 2 "Pin_Headers:Pin_Header_Straight_1x04_Pitch2.54mm" H 9250 5650 50  0001 C CNN
+F 3 "" H 9250 5650 50  0001 C CNN
+	1    9250 5650
+	0    -1   1    0
+$EndComp
+$Comp
+L CONN_01X04 J_AUX2MAIN_2
+U 1 1 5A404A42
+P 10000 5650
+F 0 "J_AUX2MAIN_2" V 10100 5650 50  0000 C CNN
+F 1 "CONN_01X04" V 10100 5650 50  0001 C CNN
+F 2 "Pin_Headers:Pin_Header_Straight_1x04_Pitch2.54mm" H 10000 5650 50  0001 C CNN
+F 3 "" H 10000 5650 50  0001 C CNN
+	1    10000 5650
+	0    -1   1    0
+$EndComp
+Wire Wire Line
+	9400 4650 9450 4650
+Wire Wire Line
+	9750 4650 9800 4650
+Wire Wire Line
+	10100 4650 10150 4650
+Wire Wire Line
+	9300 4800 9100 4800
+Wire Wire Line
+	9100 4800 9100 4850
+Wire Wire Line
+	9250 5000 9250 5000
+Wire Wire Line
+	9250 5000 9250 5150
+Wire Wire Line
+	9250 5150 9200 5150
+Wire Wire Line
+	10050 4800 9850 4800
+Wire Wire Line
+	9850 4800 9850 4850
+Wire Wire Line
+	10000 5000 10000 5150
+Wire Wire Line
+	10000 5150 9950 5150
 $EndSCHEMATC

Commit message: Updates
Parts:
- C1, C2, C3, C4, C5, C6, C7, C8, C9: footprint Capacitors_SMD:C_0805 -> Capacitors_SMD:C_0805_HandSoldering
- R1, R10, R11, R12, R13, R14, R15, R16, R2, R3, R4, R5, R6, R7, R8, R9: footprint Resistors_SMD:R_0805 -> Capacitors_SMD:C_0805_HandSoldering
Changed lines of the file:
@@
 F 0 "R1" H 3850 2050 50  0000 C CNN
 F 1 "1M" H 3850 2150 50  0000 C CNN
-F 2 "Resistors_SMD:R_0805" V 3630 2100 50  0001 C CNN
+F 2 "Capacitors_SMD:C_0805_HandSoldering" V 3630 2100 50  0001 C CNN
 F 3 "" H 3700 2100 50  0001 C CNN
 	1    3700 2100
@@
 F 0 "R3" H 4350 3400 50  0000 C CNN
 F 1 "1M" H 4350 3500 50  0000 C CNN
-F 2 "Resistors_SMD:R_0805" V 4130 3450 50  0001 C CNN
+F 2 "Capacitors_SMD:C_0805_HandSoldering" V 4130 3450 50  0001 C CNN
 F 3 "" H 4200 3450 50  0001 C CNN
 	1    4200 3450
@@
 F 0 "C1" V 3850 2950 50  0000 L CNN
 F 1 "47nF" V 4150 2950 50  0000 L CNN
-F 2 "Capacitors_SMD:C_0805" H 4038 2850 50  0001 C CNN
+F 2 "Capacitors_SMD:C_0805_HandSoldering" H 4038 2850 50  0001 C CNN
 F 3 "" H 4000 3000 50  0001 C CNN
 	1    4000 3000
@@
 F 0 "R2" H 4350 2350 50  0000 C CNN
 F 1 "1M" H 4350 2450 50  0000 C CNN
-F 2 "Resistors_SMD:R_0805" V 4130 2400 50  0001 C CNN
+F 2 "Capacitors_SMD:C_0805_HandSoldering" V 4130 2400 50  0001 C CNN
 F 3 "" H 4200 2400 50  0001 C CNN
 	1    4200 2400
@@
 F 0 "R5" H 4550 3500 50  0000 C CNN
 F 1 "10K" H 4550 3400 50  0000 C CNN
-F 2 "Resistors_SMD:R_0805" V 4630 3450 50  0001 C CNN
+F 2 "Capacitors_SMD:C_0805_HandSoldering" V 4630 3450 50  0001 C CNN
 F 3 "" H 4700 3450 50  0001 C CNN
 	1    4700 3450
@@
 F 0 "C5" V 5300 2700 50  0000 L CNN
 F 1 "10uF" V 5000 2650 50  0000 L CNN
-F 2 "Capacitors_SMD:C_0805" H 5188 2550 50  0001 C CNN
+F 2 "Capacitors_SMD:C_0805_HandSoldering" H 5188 2550 50  0001 C CNN
 F 3 "" H 5150 2700 50  0001 C CNN
 	1    5150 2700
@@
 F 0 "C6" V 5400 2650 50  0000 L CNN
 F 1 "220nF" V 5700 2600 50  0000 L CNN
-F 2 "Capacitors_SMD:C_0805" H 5588 2550 50  0001 C CNN
+F 2 "Capacitors_SMD:C_0805_HandSoldering" H 5588 2550 50  0001 C CNN
 F 3 "" H 5550 2700 50  0001 C CNN
 	1    5550 2700
@@
 F 0 "R8" H 5650 3500 50  0000 C CNN
 F 1 "150K" H 5650 3400 50  0000 C CNN
-F 2 "Resistors_SMD:R_0805" V 5730 3450 50  0001 C CNN
+F 2 "Capacitors_SMD:C_0805_HandSoldering" V 5730 3450 50  0001 C CNN
 F 3 "" H 5800 3450 50  0001 C CNN
 	1    5800 3450
@@
 F 0 "R10" V 6280 2150 50  0000 C CNN
 F 1 "4.7K" V 6200 2150 50  0000 C CNN
-F 2 "Resistors_SMD:R_0805" V 6130 2150 50  0001 C CNN
+F 2 "Capacitors_SMD:C_0805_HandSoldering" V 6130 2150 50  0001 C CNN
 F 3 "" H 6200 2150 50  0001 C CNN
 	1    6200 2150
@@
 F 0 "R7" V 5880 2250 50  0000 C CNN
 F 1 "560K" V 5800 2250 50  0000 C CNN
-F 2 "Resistors_SMD:R_0805" V 5730 2250 50  0001 C CNN
+F 2 "Capacitors_SMD:C_0805_HandSoldering" V 5730 2250 50  0001 C CNN
 F 3 "" H 5800 2250 50  0001 C CNN
 	1    5800 2250
@@
 F 0 "R11" V 6350 3000 50  0000 C CNN
 F 1 "180R" V 6550 3000 50  0000 C CNN
-F 2 "Resistors_SMD:R_0805" V 6380 3000 50  0001 C CNN
+F 2 "Capacitors_SMD:C_0805_HandSoldering" V 6380 3000 50  0001 C CNN
 F 3 "" H 6450 3000 50  0001 C CNN
 	1    6450 3000
@@
 F 0 "R12" H 6850 3400 50  0000 C CNN
 F 1 "1.2K" H 6850 3500 50  0000 C CNN
-F 2 "Resistors_SMD:R_0805" V 6630 3450 50  0001 C CNN
+F 2 "Capacitors_SMD:C_0805_HandSoldering" V 6630 3450 50  0001 C CNN
 F 3 "" H 6700 3450 50  0001 C CNN
 	1    6700 3450
@@
 F 0 "C9" V 7100 3000 50  0000 L CNN
 F 1 "10uF" V 6800 3000 50  0000 L CNN
-F 2 "Capacitors_SMD:C_0805" H 6988 2850 50  0001 C CNN
+F 2 "Capacitors_SMD:C_0805_HandSoldering" H 6988 2850 50  0001 C CNN
 F 3 "" H 6950 3000 50  0001 C CNN
 	1    6950 3000
@@
 F 0 "C7" V 6400 2350 50  0000 L CNN
 F 1 "470nF" V 6700 2350 50  0000 L CNN
-F 2 "Capacitors_SMD:C_0805" H 6588 2250 50  0001 C CNN
+F 2 "Capacitors_SMD:C_0805_HandSoldering" H 6588 2250 50  0001 C CNN
 F 3 "" H 6550 2400 50  0001 C CNN
 	1    6550 2400
@@
 F 0 "R13" V 7080 4700 50  0000 C CNN
 F 1 "68k" V 7000 4700 50  0000 C CNN
-F 2 "Resistors_SMD:R_0805" V 6930 4700 50  0001 C CNN
+F 2 "Capacitors_SMD:C_0805_HandSoldering" V 6930 4700 50  0001 C CNN
 F 3 "" H 7000 4700 50  0001 C CNN
 	1    7000 4700
@@
 F 0 "C8" V 6050 5300 50  0000 L CNN
 F 1 "470nF" V 6350 5250 50  0000 L CNN
-F 2 "Capacitors_SMD:C_0805" H 6238 5200 50  0001 C CNN
+F 2 "Capacitors_SMD:C_0805_HandSoldering" H 6238 5200 50  0001 C CNN
 F 3 "" H 6200 5350 50  0001 C CNN
 	1    6200 5350
@@
 F 0 "R6" V 5680 5350 50  0000 C CNN
 F 1 "2.2M" V 5600 5350 50  0000 C CNN
-F 2 "Resistors_SMD:R_0805" V 5530 5350 50  0001 C CNN
+F 2 "Capacitors_SMD:C_0805_HandSoldering" V 5530 5350 50  0001 C CNN
 F 3 "" H 5600 5350 50  0001 C CNN
 	1    5600 5350
@@
 F 0 "R9" H 10100 4600 50  0000 C CNN
 F 1 "10K" H 10100 4700 50  0000 C CNN
-F 2 "Resistors_SMD:R_0805" V 9880 4650 50  0001 C CNN
+F 2 "Capacitors_SMD:C_0805_HandSoldering" V 9880 4650 50  0001 C CNN
 F 3 "" H 9950 4650 50  0001 C CNN
 	1    9950 4650
@@
 F 0 "C3" V 4750 5650 50  0000 L CNN
 F 1 "1uF" V 4850 5650 50  0000 L CNN
-F 2 "Capacitors_SMD:C_0805" H 5038 5550 50  0001 C CNN
+F 2 "Capacitors_SMD:C_0805_HandSoldering" H 5038 5550 50  0001 C CNN
 F 3 "" H 5000 5700 50  0001 C CNN
 	1    5000 5700
@@
 F 0 "C4" V 4850 6050 50  0000 L CNN
 F 1 "1uF" V 4750 6050 50  0000 L CNN
-F 2 "Capacitors_SMD:C_0805" H 5038 5950 50  0001 C CNN
+F 2 "Capacitors_SMD:C_0805_HandSoldering" H 5038 5950 50  0001 C CNN
 F 3 "" H 5000 6100 50  0001 C CNN
 	1    5000 6100
@@
 F 0 "C2" H 4575 6000 50  0000 L CNN
 F 1 "1uF" H 4575 5800 50  0000 L CNN
-F 2 "Capacitors_SMD:C_0805" H 4588 5750 50  0001 C CNN
+F 2 "Capacitors_SMD:C_0805_HandSoldering" H 4588 5750 50  0001 C CNN
 F 3 "" H 4550 5900 50  0001 C CNN
 	1    4550 5900
@@
 F 0 "R4" H 4700 6300 50  0000 C CNN
 F 1 "15K" H 4700 6400 50  0000 C CNN
-F 2 "Resistors_SMD:R_0805" V 4480 6350 50  0001 C CNN
+F 2 "Capacitors_SMD:C_0805_HandSoldering" V 4480 6350 50  0001 C CNN
 F 3 "" H 4550 6350 50  0001 C CNN
 	1    4550 6350
@@
 F 0 "R15" V 7080 4300 50  0000 C CNN
 F 1 "100K" V 7000 4300 50  0000 C CNN
-F 2 "Resistors_SMD:R_0805" V 6930 4300 50  0001 C CNN
+F 2 "Capacitors_SMD:C_0805_HandSoldering" V 6930 4300 50  0001 C CNN
 F 3 "" H 7000 4300 50  0001 C CNN
 	1    7000 4300
@@
 F 0 "R14" V 6780 4300 50  0000 C CNN
 F 1 "180K" V 6700 4300 50  0000 C CNN
-F 2 "Resistors_SMD:R_0805" V 6630 4300 50  0001 C CNN
+F 2 "Capacitors_SMD:C_0805_HandSoldering" V 6630 4300 50  0001 C CNN
 F 3 "" H 6700 4300 50  0001 C CNN
 	1    6700 4300
@@
 F 0 "R16" V 4330 5700 50  0000 C CNN
 F 1 "4K7" V 4250 5700 50  0000 C CNN
-F 2 "Resistors_SMD:R_0805" V 4180 5700 50  0001 C CNN
+F 2 "Capacitors_SMD:C_0805_HandSoldering" V 4180 5700 50  0001 C CNN
 F 3 "" H 4250 5700 50  0001 C CNN
 	1    4250 5700
