File: EATremoloSMD/EATremoloSMD.sch (KiCad schematic (older format))
At the start: 42 parts, among them J1 JACK__MONO_2P_NC, J2 BARREL_JACK, J3 JACK__MONO_2P_NC, Q1 Q_NJFET_DSG, Q2 Q_NPN_EBC, Q3 Q_NPN_EBC, Q4 Q_NJFET_DSG, SW1 SW_3PDT_on_on

Commit message: update
Parts:
- R16: value 1K8 -> 2K4
- R4: value 18K -> 12K
- R6: value 2.2M -> 1.2M
- RATE1: value B100K -> B10K
Changed lines of the file:
@@
 P 5600 5350
 F 0 "R6" V 5680 5350 50  0000 C CNN
-F 1 "2.2M" V 5600 5350 50  0000 C CNN
+F 1 "1.2M" V 5600 5350 50  0000 C CNN
 F 2 "Capacitors_SMD:C_0805_HandSoldering" V 5530 5350 50  0001 C CNN
 F 3 "" H 5600 5350 50  0001 C CNN
@@
 P 4550 6350
 F 0 "R4" H 4700 6300 50  0000 C CNN
-F 1 "18K" H 4700 6400 50  0000 C CNN
+F 1 "12K" H 4700 6400 50  0000 C CNN
 F 2 "Capacitors_SMD:C_0805_HandSoldering" V 4480 6350 50  0001 C CNN
 F 3 "" H 4550 6350 50  0001 C CNN
@@
 P 9100 5000
 F 0 "RATE1" V 8925 5000 50  0000 C CNN
-F 1 "B100K" V 9000 5000 50  0000 C CNN
+F 1 "B10K" V 9000 5000 50  0000 C CNN
 F 2 "Potentiometers:Potentiometer_Bourns_PTV09A-1_Horizontal" H 9100 5000 50  0001 C CNN
 F 3 "" H 9100 5000 50  0001 C CNN
@@
 P 3775 5700
 F 0 "R16" V 3855 5700 50  0000 C CNN
-F 1 "1K8" V 3775 5700 50  0000 C CNN
+F 1 "2K4" V 3775 5700 50  0000 C CNN
 F 2 "Capacitors_SMD:C_0805_HandSoldering" V 3705 5700 50  0001 C CNN
 F 3 "" H 3775 5700 50  0001 C CNN
