File: HexTremolo/HexTremolo/HexTremolo.sch (KiCad schematic (older format))
At the start: 23 parts, among them U5 4N35

Commit message: update
Parts:
- added C4: 22uF, symbol Device:CP
- added R10, R9: 100R, symbol Device:R
- added R8: 560R, symbol Device:R
Connections:
- wire segments 106 -> 113
Other:
- moved on the sheet: J_PWR1, U5, U_BUF1A, U_BUF1B, U_BUF1C

Commit message: UPDATED SCHEMATIC
removed clk tick from audio path
- current limiting resistors at osc vcc (1W)
- LPF at FX-side of OPTOCOUPLER
Parts:
- removed R10: 100R, symbol Device:R
- removed R7: 10K, symbol Device:R
- added C_BP1, C_BP2, C_BP3, C_BP4, C_BP5: 100nF, symbol Device:C
- added R_OSC1: 1K, symbol Device:R
- added SW_MODE1: SW_SPDT, symbol Switch:SW_SPDT
- added U? (x4): 74HC7014, Package_SO:SOIC-14_3.9x8.7mm_P1.27mm, symbol 74xx:74HC7014
- C1, C2: value CP -> 10uF
- C_LPF1: renamed from C4; value 22uF -> 10uF
- C_OSC1: renamed from C3; value 47uF -> 22uF
- P_DEPTH1: renamed from DEPTH1; value B10k -> B100k
- P_RATE1: renamed from SPEED1; value B100K -> B10K
- R9: value 100R -> 200R 1W
- R_GAIN1: renamed from R6; value 1K -> 3K9
- R_LPF1: renamed from R8; value 560R -> 100R
- renumbered D1 to D_LED1, VOLUME1 to P_VOL1, U5 to U_OPTO1
Connections:
- wire segments 113 -> 141
- no-connect marks 2 -> 10
Other:
- moved on the sheet: J_PWR1, U_BUF1A, U_BUF1B, U_OPTO1

Commit message: RevA
Parts:
- removed C_LPF1: 10uF, symbol Device:CP
- removed C_OSC1: 22uF, symbol Device:CP
- removed D_LED1: LED, symbol Device:LED
- removed J_IN1, J_OUT1: AudioJack2_Ground_Switch, symbol Connector:AudioJack2_Ground_Switch
- removed P_RATE1: B10K, symbol Device:R_POT
- removed R9: 200R 1W, symbol Device:R
- removed R_LPF1: 100R, symbol Device:R
- removed R_OSC1: 1K, symbol Device:R
- removed SW_MODE1: SW_SPDT, symbol Switch:SW_SPDT
- removed U? (x4): 74HC7014, Package_SO:SOIC-14_3.9x8.7mm_P1.27mm, symbol 74xx:74HC7014
- removed U_NREG1: LM337_TO220, Package_TO_SOT_THT:TO-220-3_Vertical, symbol Regulator_Linear:LM337_TO220
- removed U_OPTO1: 4N35, Package_DIP:DIP-6_W7.62mm, symbol Isolator:4N35
- removed unit 1 of U_OSC1
- removed unit 2 of U_OSC1
- added J_IN1, J_OUT1: JACK__MONO_2P_NC, custom_sockets:6_35MM_JACK_MONO_FlatTop, symbol socket_custom:JACK__MONO_2P_NC
- added R6: 200R 1W, Resistor_SMD:R_0805_2012Metric_Pad1.15x1.40mm_HandSolder, symbol Device:R
- added U_NREG1: LM337_SOT223, Package_TO_SOT_SMD:SOT-223-3_TabPin2, symbol Regulator_Linear:LM337_SOT223
- added unit 3 of U_OSC1
- added unit 4 of U_OSC1
- added unit 5 of U_OSC1
- added unit 6 of U_OSC1
- CP_INV1: renamed from C1; footprint (none) -> Capacitor_SMD:CP_Elec_4x5.4
- CP_INV2: renamed from C2; footprint (none) -> Capacitor_SMD:CP_Elec_4x5.4
- C_BP1, C_BP2, C_BP3, C_BP4, C_BP5: footprint (none) -> Capacitor_SMD:C_0805_2012Metric_Pad1.15x1.40mm_HandSolder
- J_PWR1: footprint (none) -> Connector_BarrelJack:BarrelJack_Horizontal
- P_DEPTH1: value B100k -> B50k; footprint (none) -> Potentiometer_THT:Potentiometer_Alps_RK09L_Single_Vertical
- P_VOL1: footprint (none) -> Potentiometer_THT:Potentiometer_Alps_RK09L_Single_Vertical
- R1, R2, R3, R4, R5, R_GAIN1: footprint (none) -> Resistor_SMD:R_0805_2012Metric_Pad1.15x1.40mm_HandSolder
- U_BUF1: footprint (none) -> Package_SO:SOIC-8_3.9x4.9mm_P1.27mm
- U_PREG1: footprint (none) -> Package_TO_SOT_SMD:SOT-223-3_TabPin2
Connections:
- net labels added: 3PDT_2_EXT, 3PDT_3_EXT, 3PDT_4_EXT, 3PDT_5_EXT, 3PDT_6_EXT, 3PDT_8_EXT, 3PDT__1_EXT
- wire segments 141 -> 126
Other:
- note added: "BYPASS"
- note added: "POWER SUPPLY"
- moved on the sheet: J_PWR1, U_BUF1A, U_BUF1B, U_BUF1C
