File: HexTremolo/HexTremolo/HexInverter_3PDT.sch (KiCad schematic (older format))
At the start: 3 parts

Commit message: RevA
Parts:
- removed J_AUXTOMAIN1, J_MAINTOAUX1: Conn_01x10, Connector_PinHeader_1.27mm:PinHeader_1x10_P1.27mm_Vertical, symbol Connector_Generic:Conn_01x10
- added J_AUXTOMAIN1, J_MAINTOAUX1: Conn_01x09, Connector_PinHeader_1.27mm:PinHeader_1x09_P1.27mm_Vertical, symbol Connector_Generic:Conn_01x09
Connections:
- no-connect marks 2 -> 0
Changed lines of the file:
@@
 	1    0    0    -1
 $EndComp
-Text HLabel 3350 3250 0    50   Input ~ 0
+Text HLabel 3200 3200 0    50   Input ~ 0
 3PDT_2
-Text HLabel 3350 3550 0    50   Input ~ 0
+Text HLabel 3200 3500 0    50   Input ~ 0
 3PDT_5
-Text HLabel 3350 3750 0    50   Input ~ 0
+Text HLabel 3200 3700 0    50   Input ~ 0
 3PDT_7
-Text HLabel 3350 3850 0    50   Input ~ 0
+Text HLabel 3200 3800 0    50   Input ~ 0
 3PDT_8
-Text HLabel 3350 3950 0    50   Input ~ 0
+Text HLabel 3200 3900 0    50   Input ~ 0
 3PDT_9
-Text HLabel 3350 3650 0    50   Input ~ 0
+Text HLabel 3200 3600 0    50   Input ~ 0
 3PDT_6
-Text HLabel 3350 3450 0    50   Input ~ 0
+Text HLabel 3200 3400 0    50   Input ~ 0
 3PDT_4
-Text HLabel 3350 3350 0    50   Input ~ 0
+Text HLabel 3200 3300 0    50   Input ~ 0
 3PDT_3
-Text HLabel 3350 3150 0    50   Input ~ 0
+Text HLabel 3200 3100 0    50   Input ~ 0
 3PDT_1
 Wire Wire Line
-	3350 3250 3750 3250
+	3200 3200 3600 3200
 Wire Wire Line
-	3750 3550 3350 3550
+	3600 3500 3200 3500
 Wire Wire Line
-	3350 3850 3750 3850
+	3200 3800 3600 3800
 Wire Wire Line
-	3750 3950 3350 3950
+	3600 3900 3200 3900
 Wire Wire Line
-	3350 3750 3750 3750
+	3200 3700 3600 3700
 Wire Wire Line
-	3750 3650 3350 3650
+	3600 3600 3200 3600
 Wire Wire Line
-	3350 3450 3750 3450
+	3200 3400 3600 3400
 Wire Wire Line
-	3750 3350 3350 3350
+	3600 3300 3200 3300
 Wire Wire Line
-	3350 3150 3750 3150
-$Comp
-L Connector_Generic:Conn_01x10 J_MAINTOAUX1
-U 1 1 5BFD031D
-P 3950 3550
-F 0 "J_MAINTOAUX1" H 3550 4200 50  0000 L CNN
-F 1 "Conn_01x10" H 3600 4100 50  0000 L CNN
-F 2 "Connector_PinHeader_1.27mm:PinHeader_1x10_P1.27mm_Vertical" H 3950 3550 50  0001 C CNN
-F 3 "~" H 3950 3550 50  0001 C CNN
-	1    3950 3550
-	1    0    0    -1
-$EndComp
-$Comp
-L Connector_Generic:Conn_01x10 J_AUXTOMAIN1
-U 1 1 5BFD0349
-P 4400 3550
-F 0 "J_AUXTOMAIN1" H 4300 4200 50  0000 C CNN
-F 1 "Conn_01x10" H 4300 4100 50  0000 C CNN
-F 2 "Connector_PinHeader_1.27mm:PinHeader_1x10_P1.27mm_Vertical" H 4400 3550 50  0001 C CNN
-F 3 "~" H 4400 3550 50  0001 C CNN
-	1    4400 3550
-	-1   0    0    -1
-$EndComp
-NoConn ~ 3750 4050
+	3200 3100 3600 3100
 Wire Wire Line
-	4600 3150 5050 3150
+	4450 3100 5100 3100
 Wire Wire Line
-	4600 3250 5050 3250
+	4450 3200 5100 3200
 Wire Wire Line
-	4600 3350 5050 3350
+	4450 3300 5100 3300
 Wire Wire Line
-	4600 3450 5050 3450
+	4450 3400 5100 3400
 Wire Wire Line
-	4600 3550 5050 3550
+	4450 3500 5100 3500
 Wire Wire Line
-	4600 3650 5050 3650
+	4450 3600 5100 3600
 Wire Wire Line
-	4600 3750 5050 3750
+	4450 3700 5100 3700
 Wire Wire Line
-	4600 3850 5050 3850
+	4450 3800 5100 3800
 Wire Wire Line
-	4600 3950 5050 3950
-NoConn ~ 4600 4050
+	4450 3900 5100 3900
 Wire Wire Line
 	6450 2950 6150 2950
@@
 Wire Wire Line
 	6850 2850 7150 2850
-Text Label 5050 3150 2    50   ~ 0
+Text Label 5100 3100 2    50   ~ 0
 3PDT_1_INT
-Text Label 5050 3250 2    50   ~ 0
+Text Label 5100 3200 2    50   ~ 0
 3PDT_2_INT
-Text Label 5050 3350 2    50   ~ 0
+Text Label 5100 3300 2    50   ~ 0
 3PDT_3_INT
-Text Label 5050 3450 2    50   ~ 0
+Text Label 5100 3400 2    50   ~ 0
 3PDT_4_INT
-Text Label 5050 3550 2    50   ~ 0
+Text Label 5100 3500 2    50   ~ 0
 3PDT_5_INT
-Text Label 5050 3650 2    50   ~ 0
+Text Label 5100 3600 2    50   ~ 0
 3PDT_6_INT
-Text Label 5050 3750 2    50   ~ 0
+Text Label 5100 3700 2    50   ~ 0
 3PDT_7_INT
-Text Label 5050 3850 2    50   ~ 0
+Text Label 5100 3800 2    50   ~ 0
 3PDT_8_INT
-Text Label 5050 3950 2    50   ~ 0
+Text Label 5100 3900 2    50   ~ 0
 3PDT_9_INT
 Text Label 6150 2950 2    50   ~ 0
@@
 Text Label 7150 4250 0    50   ~ 0
 3PDT_9_INT
+$Comp
+L Connector_Generic:Conn_01x09 J_MAINTOAUX1
+U 1 1 5BE491D7
+P 3800 3500
+F 0 "J_MAINTOAUX1" H 3350 4150 50  0000 L CNN
+F 1 "Conn_01x09" H 3400 4050 50  0000 L CNN
+F 2 "Connector_PinHeader_1.27mm:PinHeader_1x09_P1.27mm_Vertical" H 3800 3500 50  0001 C CNN
+F 3 "~" H 3800 3500 50  0001 C CNN
+	1    3800 3500
+	1    0    0    -1
+$EndComp
+$Comp
+L Connector_Generic:Conn_01x09 J_AUXTOMAIN1
+U 1 1 5BE49202
+P 4250 3500
+F 0 "J_AUXTOMAIN1" H 4150 4150 50  0000 C CNN
+F 1 "Conn_01x09" H 4150 4050 50  0000 C CNN
+F 2 "Connector_PinHeader_1.27mm:PinHeader_1x09_P1.27mm_Vertical" H 4250 3500 50  0001 C CNN
+F 3 "~" H 4250 3500 50  0001 C CNN
+	1    4250 3500
+	-1   0    0    -1
+$EndComp
 $EndSCHEMATC
