File: HexTremolo/HexTremolo/HexInverter_Clock.sch (KiCad schematic (older format))
At the start: 11 parts

Commit message: RevA
Parts:
- U_OPTO1: footprint Package_DIP:SMDIP-6_W9.53mm -> Package_DIP:SMDIP-6_W7.62mm
Changed lines of the file:
@@
 F 0 "U_OPTO1" V 8750 3350 50  0000 R CNN
 F 1 "4N35" V 8650 3300 50  0000 R CNN
-F 2 "Package_DIP:SMDIP-6_W9.53mm" H 8500 2600 50  0001 L CIN
+F 2 "Package_DIP:SMDIP-6_W7.62mm" H 8500 2600 50  0001 L CIN
 F 3 "https://www.vishay.com/docs/81181/4n35.pdf" H 8700 2800 50  0001 L CNN
 	1    8700 2800
