File: HexTremolo/HexTremolo/HexTremolo.kicad_pcb (KiCad board)
At the start: 2 copper layers, 56.4 x 96 mm, 37 parts

Commit message: RevA
Parts:
- J_AUXTOMAIN1, J_MAINTOAUX1: value Conn_01x10 -> Conn_01x09; footprint Connector_PinHeader_1.27mm:PinHeader_1x10_P1.27mm_Vertical -> Connector_PinHeader_1.27mm:PinHeader_1x09_P1.27mm_Vertical
- moved C_BP4 2.54 mm to (105.7, 124.0)
- moved U_BUF1 2.54 mm to (101.6, 120.1)
- moved C_BP3 2.54 mm to (99.7, 113.0)
- moved J_AUXTOMAIN1 2.54 mm to (101.6, 147.3)
- moved J_MAINTOAUX1 2.54 mm to (101.6, 130.6)
- moved R_GAIN1 2.54 mm to (102.2, 113.0)
- moved R3 1.30 mm to (72.8, 118.2)
- moved R4 1.30 mm to (72.8, 123.3)
- moved R5 1.30 mm to (72.8, 120.8)
- moved U_NREG1 1.30 mm to (80.5, 120.8)
- moved SW_EN1 1.05 mm to (80.5, 157.5)
- moved CP_INV1 0.77 mm to (56.6, 131.8)
Routing:
- net -5V: track 49.9 -> 60.8 mm
- net /3PDT_8_EXT: track 79.8 -> 86.8 mm
- net /3PDT_5_EXT: track 54.0 -> 60.9 mm
- net /3PDT_3_EXT: track 13.4 -> 18.6 mm
- net /HexInverter_3PDT/3PDT_6_INT: track 16.0 -> 19.7 mm
- net /3PDT_2_EXT: track 23.9 -> 27.4 mm
- net -9V: track 47.8 -> 44.4 mm, vias 0 -> 12
- net Net-(P_DEPTH1-Pad1): track 78.9 -> 76.1 mm
- net +5V: track 128.2 -> 131.0 mm, vias 3 -> 15
- net /HexInverter_3PDT/3PDT_8_INT: track 23.8 -> 26.4 mm
- net /HexInverter_3PDT/3PDT_7_INT: track 42.6 -> 44.7 mm
- net /HexInverter_3PDT/3PDT_3_INT: track 14.2 -> 15.7 mm
- net /HexInverter_3PDT/3PDT_1_INT: track 24.1 -> 25.3 mm
- net /HexInverter_3PDT/3PDT_2_INT: track 19.0 -> 20.1 mm
- net Net-(P_VOL1-Pad1): track 62.1 -> 60.9 mm
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- added copper zone on B.Cu, net +5V
- added copper zone on B.Cu, net -9V
Other:
- outline, holes or cut-outs redrawn
