File: 555PWMTremolo/555PWMTremolo.kicad_pcb (KiCad board)
At the start: 2 copper layers, 54.6 x 98.6 mm, 37 parts

Commit message: Final RevA
Parts:
- removed CP_LPF1: 22uF, Capacitor_SMD:CP_Elec_4x5.4
- added CP_FAST1: 22uF, Capacitor_SMD:CP_Elec_4x5.4, F.Cu at (83.6, 91.4)
- added CP_SLOW1: 220uF, Capacitor_SMD:CP_Elec_6.3x5.4, F.Cu at (95.2, 90.7)
- added R_OSCLIMIT1: 100R, Resistor_SMD:R_0805_2012Metric_Pad1.15x1.40mm_HandSolder, B.Cu at (66.0, 104.9)
- added SW_ATTACK1: SW_SPDT, DailywellSwitches:Dailywell_SPDT, F.Cu at (80.6, 85.3)
- C_BP1, C_BP3, C_BP4, C_OSC2: moved to F.Cu
- C_LPFOPT1, C_LPFOPT2, R_LPF1: moved to B.Cu
- moved C_BP5 18.8 mm to (56.6, 136.9), turned to 0 degrees
- moved D_LED1 8.75 mm to (82.0, 97.5), turned to 180 degrees
- moved R_OSCOFF1 6.36 mm to (65.0, 94.7), turned to 180 degrees
- moved R1 5.41 mm to (75.0, 135.5)
- moved C_LPFOPT2 4.62 mm to (84.5, 79.2), turned to 270 degrees
- moved R_LPF1 4.59 mm to (80.6, 79.2)
- moved C_LPFOPT1 4.57 mm to (76.8, 79.2), turned to 270 degrees
- moved U_OPTO1 2.54 mm to (80.6, 74.3)
- moved C_BP4 2.45 mm to (81.5, 116.7), turned to 270 degrees
- moved R2 1.98 mm to (83.6, 135.4)
- moved C_BP3 1.94 mm to (77.7, 104.5), turned to 270 degrees
- moved C_OSC2 1.44 mm to (71.0, 93.0), turned to 270 degrees
- moved J_MAINTOAUX1 1.27 mm to (87.0, 128.0)
- moved U_NREG1 0.76 mm to (97.1, 141.9)
- moved U_PREG1 0.76 mm to (80.6, 141.4)
Connections:
- C_BP1 pad 1: /3PDT_8_EXT -> Net-(C_BP1-Pad1)
- R_OSCOFF1 pad 2: /3PDT_8_EXT -> Net-(C_BP1-Pad1)
- U_OSC1 pad 4: /3PDT_8_EXT -> Net-(C_BP1-Pad1)
- U_OSC1 pad 8: /3PDT_8_EXT -> Net-(C_BP1-Pad1)
Routing:
- net /3PDT_8_EXT: track 108.6 -> 40.4 mm
- net Net-(C_BP1-Pad1): track 0.00 -> 57.4 mm, vias 0 -> 1
- net Net-(C_LPFOPT1-Pad1): track 13.8 -> 29.2 mm, vias 0 -> 1
- net Net-(CP_SLOW1-Pad1): track 0.00 -> 12.1 mm
- net Net-(P_DEPTH1-Pad2): track 32.1 -> 44.1 mm
- net Net-(CP_FAST1-Pad1): track 0.00 -> 8.08 mm
- net +5V: track 101.0 -> 93.8 mm, vias 19 -> 16
- net /GND: track 20.7 -> 25.8 mm, vias 11 -> 15
- net Net-(P_OSCOFF1-Pad1): track 10.2 -> 5.57 mm
- net Net-(C_LPFOPT2-Pad1): track 39.9 -> 43.5 mm, vias 0 -> 1
- net +9V: track 29.1 -> 25.7 mm
- net /555PWMTremolo_Clock/CLK_OUT: track 16.7 -> 19.2 mm
- net Net-(P_OSCOFF1-Pad3): track 18.7 -> 20.0 mm
- net /3PDT_2_EXT: track 8.91 -> 10.1 mm
- net -9V: track 46.5 -> 47.6 mm
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
Commit message: Final RevA
Other:
- board text added: "OPTO TREM Chris Sutton 2018 RevA"
- board text added: "OPTO TREM Chris Sutton RevA 2018"
Changed lines of the file:
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@@
   (general
     (thickness 1.6)
-    (drawings 18)
+    (drawings 20)
     (tracks 397)
     (zones 0)
@@
       (rotate (xyz 0 0 90))
     )
+  )
+  (gr_text "OPTO TREM\nChris Sutton\nRevA 2018" (at 99.187 131.191) (layer B.SilkS)
+    (effects (font (size 1 1) (thickness 0.2)) (justify mirror))
+  )
+  (gr_text "OPTO TREM\nChris Sutton\n2018 RevA" (at 65.532 159.766) (layer B.SilkS)
+    (effects (font (size 1 1) (thickness 0.2)) (justify mirror))
   )
   (gr_line (start 53.34 72.39) (end 54.356 71.374) (layer Edge.Cuts) (width 0.2))
@@
   (segment (start 76.962 97.536) (end 76.2 96.774) (width 0.25) (layer F.Cu) (net 19))
   (segment (start 79.502 97.536) (end 76.962 97.536) (width 0.25) (layer F.Cu) (net 19))
-  (via (at 84.455 76.835) (size 0.8) (drill 0.4) (layers F.Cu B.Cu) (net 38))
-  (segment (start 84.455 76.835) (end 82.55 76.835) (width 0.25) (layer F.Cu) (net 38))
-  (segment (start 82.55 76.835) (end 79.375 73.66) (width 0.25) (layer F.Cu) (net 38))
-  (segment (start 79.375 73.66) (end 77.495 73.66) (width 0.25) (layer F.Cu) (net 38))
   (segment (start 59.839 140.771) (end 59.784 140.716) (width 0.5) (layer F.Cu) (net 20))
   (segment (start 59.839 144.526) (end 59.839 140.771) (width 0.5) (layer F.Cu) (net 20))
@@
   (segment (start 66.04 100.076) (end 70.358 100.076) (width 0.75) (layer F.Cu) (net 37))
   (segment (start 67.724 88.138) (end 70.993 88.138) (width 0.5) (layer F.Cu) (net 37))
+  (via (at 84.455 76.835) (size 0.8) (drill 0.4) (layers F.Cu B.Cu) (net 38))
+  (segment (start 84.455 76.835) (end 82.55 76.835) (width 0.25) (layer F.Cu) (net 38))
+  (segment (start 82.55 76.835) (end 79.375 73.66) (width 0.25) (layer F.Cu) (net 38))
+  (segment (start 79.375 73.66) (end 77.495 73.66) (width 0.25) (layer F.Cu) (net 38))
   (segment (start 84.582 78.223) (end 84.455 78.096) (width 0.25) (layer B.Cu) (net 38))
   (segment (start 84.455 76.835) (end 84.455 78.223) (width 0.25) (layer B.Cu) (net 38))

Commit message: Final RevA
Parts:
- J_MAINTOAUX1: footprint CustomHeaders:IDCHeader_02x05_P2.54mm_Vertical_Counter_Clockwise -> CustomHeaders:IDCHeader_02x05_P2.54mm_Vertical_Clockwise; moved to B.Cu
- moved J_MAINTOAUX1 3.18 mm to (87.0, 131.2), turned to 90 degrees
- moved R2 0.25 mm to (83.6, 135.6)
- moved R1 0.15 mm to (75.0, 135.6)
Routing:
- net /3PDT_8_EXT: track 40.4 -> 42.8 mm
- net +5V: track 93.8 -> 96.2 mm
- net /3PDT_6_EXT: track 70.8 -> 72.0 mm
- net /3PDT_5_EXT: track 18.3 -> 19.1 mm
- net /3PDT_2_EXT: track 10.1 -> 10.7 mm
- net /3PDT_3_EXT: track 15.8 -> 16.4 mm

Commit message: Final RevA
Parts:
- moved C_BP3 1.02 mm to (77.7, 103.5)
Routing:
- net Net-(R_LPF1-Pad2): track 41.4 -> 42.8 mm
- net Net-(C_LPFOPT1-Pad1): track 29.2 -> 28.2 mm
- net +5V: track 96.2 -> 97.1 mm
Other:
- board text added: ">"
- board text added: "Jumper if not req’d"
- board text added: "PLUG THIS SIDE"
- board text added: "higher val lower range"
- board text added: "lower val more gain"
