File: 555PWMTremolo/555PWMTremolo_3PDT.sch (KiCad schematic (older format))
At the start: 3 parts

Commit message: Tidied up 555 layout
Parts:
- removed J_AUXTOMAIN1, J_MAINTOAUX1: Conn_01x09, Connector_PinHeader_1.27mm:PinHeader_1x09_P1.27mm_Vertical, symbol Connector_Generic:Conn_01x09
- added J_AUXTOMAIN1, J_MAINTOAUX1: Conn_02x05_Counter_Clockwise, CustomHeaders:IDCHeader_02x05_P2.54mm_Vertical_Counter_Clockwise, symbol Connector_Generic:Conn_02x05_Counter_Clockwise
Changed lines of the file:
@@
 	1    0    0    -1
 $EndComp
-Text HLabel 3200 3200 0    50   Input ~ 0
+Text HLabel 2900 4500 0    50   Input ~ 0
 3PDT_2
-Text HLabel 3200 3500 0    50   Input ~ 0
+Text HLabel 2900 4800 0    50   Input ~ 0
 3PDT_5
-Text HLabel 3200 3700 0    50   Input ~ 0
+Text HLabel 3600 4700 2    50   Input ~ 0
 3PDT_7
-Text HLabel 3200 3800 0    50   Input ~ 0
+Text HLabel 3600 4600 2    50   Input ~ 0
 3PDT_8
-Text HLabel 3200 3900 0    50   Input ~ 0
+Text HLabel 3600 4500 2    50   Input ~ 0
 3PDT_9
-Text HLabel 3200 3600 0    50   Input ~ 0
+Text HLabel 3600 4800 2    50   Input ~ 0
 3PDT_6
-Text HLabel 3200 3400 0    50   Input ~ 0
+Text HLabel 2900 4700 0    50   Input ~ 0
 3PDT_4
-Text HLabel 3200 3300 0    50   Input ~ 0
+Text HLabel 2900 4600 0    50   Input ~ 0
 3PDT_3
-Text HLabel 3200 3100 0    50   Input ~ 0
+Text HLabel 2900 4400 0    50   Input ~ 0
 3PDT_1
 Wire Wire Line
-	3200 3200 3600 3200
+	2900 4500 3000 4500
 Wire Wire Line
-	3600 3500 3200 3500
+	3000 4800 2900 4800
 Wire Wire Line
-	3200 3800 3600 3800
+	3600 4600 3500 4600
 Wire Wire Line
-	3600 3900 3200 3900
+	3500 4500 3600 4500
 Wire Wire Line
-	3200 3700 3600 3700
+	3600 4700 3500 4700
 Wire Wire Line
-	3600 3600 3200 3600
+	3500 4800 3600 4800
 Wire Wire Line
-	3200 3400 3600 3400
+	2900 4700 3000 4700
 Wire Wire Line
-	3600 3300 3200 3300
+	3000 4600 2900 4600
 Wire Wire Line
-	3200 3100 3600 3100
+	2900 4400 3000 4400
 Wire Wire Line
-	4450 3100 5100 3100
+	4800 4400 4150 4400
 Wire Wire Line
-	4450 3200 5100 3200
+	4800 4500 4150 4500
 Wire Wire Line
-	4450 3300 5100 3300
+	4800 4600 4150 4600
 Wire Wire Line
-	4450 3400 5100 3400
+	4800 4700 4150 4700
 Wire Wire Line
-	4450 3500 5100 3500
+	4800 4800 4150 4800
 Wire Wire Line
-	4450 3600 5100 3600
+	5300 4800 5800 4800
 Wire Wire Line
-	4450 3700 5100 3700
+	5300 4700 5800 4700
 Wire Wire Line
-	4450 3800 5100 3800
+	5300 4600 5800 4600
 Wire Wire Line
-	4450 3900 5100 3900
+	5300 4500 5800 4500
 Wire Wire Line
 	6450 2950 6150 2950
@@
 Wire Wire Line
 	6850 2850 7150 2850
-Text Label 5100 3100 2    50   ~ 0
+Text Label 4150 4400 0    50   ~ 0
 3PDT_1_INT
-Text Label 5100 3200 2    50   ~ 0
+Text Label 4150 4500 0    50   ~ 0
 3PDT_2_INT
-Text Label 5100 3300 2    50   ~ 0
+Text Label 4150 4600 0    50   ~ 0
 3PDT_3_INT
-Text Label 5100 3400 2    50   ~ 0
+Text Label 4150 4700 0    50   ~ 0
 3PDT_4_INT
-Text Label 5100 3500 2    50   ~ 0
+Text Label 4150 4800 0    50   ~ 0
 3PDT_5_INT
-Text Label 5100 3600 2    50   ~ 0
+Text Label 5800 4800 2    50   ~ 0
 3PDT_6_INT
-Text Label 5100 3700 2    50   ~ 0
+Text Label 5800 4700 2    50   ~ 0
 3PDT_7_INT
-Text Label 5100 3800 2    50   ~ 0
+Text Label 5800 4600 2    50   ~ 0
 3PDT_8_INT
-Text Label 5100 3900 2    50   ~ 0
+Text Label 5800 4500 2    50   ~ 0
 3PDT_9_INT
 Text Label 6150 2950 2    50   ~ 0
@@
 3PDT_9_INT
 $Comp
-L Connector_Generic:Conn_01x09 J_MAINTOAUX1
-U 1 1 5BE491D7
-P 3800 3500
-F 0 "J_MAINTOAUX1" H 3350 4150 50  0000 L CNN
-F 1 "Conn_01x09" H 3400 4050 50  0000 L CNN
-F 2 "Connector_PinHeader_1.27mm:PinHeader_1x09_P1.27mm_Vertical" H 3800 3500 50  0001 C CNN
-F 3 "~" H 3800 3500 50  0001 C CNN
-	1    3800 3500
+L Connector_Generic:Conn_02x05_Counter_Clockwise J_MAINTOAUX1
+U 1 1 5BE5C9F1
+P 3200 4600
+F 0 "J_MAINTOAUX1" H 3250 4925 50  0000 C CNN
+F 1 "Conn_02x05_Counter_Clockwise" H 3250 4926 50  0001 C CNN
+F 2 "CustomHeaders:IDCHeader_02x05_P2.54mm_Vertical_Counter_Clockwise" H 3200 4600 50  0001 C CNN
+F 3 "~" H 3200 4600 50  0001 C CNN
+	1    3200 4600
 	1    0    0    -1
 $EndComp
 $Comp
-L Connector_Generic:Conn_01x09 J_AUXTOMAIN1
-U 1 1 5BE49202
-P 4250 3500
-F 0 "J_AUXTOMAIN1" H 4150 4150 50  0000 C CNN
-F 1 "Conn_01x09" H 4150 4050 50  0000 C CNN
-F 2 "Connector_PinHeader_1.27mm:PinHeader_1x09_P1.27mm_Vertical" H 4250 3500 50  0001 C CNN
-F 3 "~" H 4250 3500 50  0001 C CNN
-	1    4250 3500
-	-1   0    0    -1
+L Connector_Generic:Conn_02x05_Counter_Clockwise J_AUXTOMAIN1
+U 1 1 5BE5CA85
+P 5000 4600
+F 0 "J_AUXTOMAIN1" H 5050 4925 50  0000 C CNN
+F 1 "Conn_02x05_Counter_Clockwise" H 5050 4926 50  0001 C CNN
+F 2 "CustomHeaders:IDCHeader_02x05_P2.54mm_Vertical_Counter_Clockwise" H 5000 4600 50  0001 C CNN
+F 3 "~" H 5000 4600 50  0001 C CNN
+	1    5000 4600
+	1    0    0    -1
 $EndComp
 $EndSCHEMATC

Commit message: Final RevA
Changed lines of the file:
@@
 L sw_custom:SW_3PDT_on_on SW_EN1
 U 1 1 5BFCF869
-P 6650 2950
-F 0 "SW_EN1" H 6650 3235 50  0000 C CNN
-F 1 "SW_3PDT_on_on" H 6650 3144 50  0000 C CNN
-F 2 "custom_sw:SW_3PDT_W18MM_L17.3MM_P5.3MM_D2MM" H 6650 2950 50  0001 C CNN
-F 3 "https://www.mouser.co.uk/datasheet/2/140/FS5700-1147045.pdf" H 6650 2950 50  0001 C CNN
-	1    6650 2950
+P 8300 2900
+F 0 "SW_EN1" H 8300 3185 50  0000 C CNN
+F 1 "SW_3PDT_on_on" H 8300 3094 50  0000 C CNN
+F 2 "custom_sw:SW_3PDT_W18MM_L17.3MM_P5.3MM_D2MM" H 8300 2900 50  0001 C CNN
+F 3 "https://www.mouser.co.uk/datasheet/2/140/FS5700-1147045.pdf" H 8300 2900 50  0001 C CNN
+	1    8300 2900
 	1    0    0    -1
 $EndComp
@@
 L sw_custom:SW_3PDT_on_on SW_EN1
 U 2 1 5BFCF8CC
-P 6650 3550
-F 0 "SW_EN1" H 6650 3835 50  0000 C CNN
-F 1 "SW_3PDT_on_on" H 6650 3744 50  0000 C CNN
-F 2 "custom_sw:SW_3PDT_W18MM_L17.3MM_P5.3MM_D2MM" H 6650 3550 50  0001 C CNN
-F 3 "https://www.mouser.co.uk/datasheet/2/140/FS5700-1147045.pdf" H 6650 3550 50  0001 C CNN
-	2    6650 3550
+P 8300 3500
+F 0 "SW_EN1" H 8300 3785 50  0000 C CNN
+F 1 "SW_3PDT_on_on" H 8300 3694 50  0000 C CNN
+F 2 "custom_sw:SW_3PDT_W18MM_L17.3MM_P5.3MM_D2MM" H 8300 3500 50  0001 C CNN
+F 3 "https://www.mouser.co.uk/datasheet/2/140/FS5700-1147045.pdf" H 8300 3500 50  0001 C CNN
+	2    8300 3500
 	1    0    0    -1
 $EndComp
@@
 L sw_custom:SW_3PDT_on_on SW_EN1
 U 3 1 5BFCF92E
-P 6650 4150
-F 0 "SW_EN1" H 6650 4435 50  0000 C CNN
-F 1 "SW_3PDT_on_on" H 6650 4344 50  0000 C CNN
-F 2 "custom_sw:SW_3PDT_W18MM_L17.3MM_P5.3MM_D2MM" H 6650 4150 50  0001 C CNN
-F 3 "https://www.mouser.co.uk/datasheet/2/140/FS5700-1147045.pdf" H 6650 4150 50  0001 C CNN
-	3    6650 4150
+P 8300 4100
+F 0 "SW_EN1" H 8300 4385 50  0000 C CNN
+F 1 "SW_3PDT_on_on" H 8300 4294 50  0000 C CNN
+F 2 "custom_sw:SW_3PDT_W18MM_L17.3MM_P5.3MM_D2MM" H 8300 4100 50  0001 C CNN
+F 3 "https://www.mouser.co.uk/datasheet/2/140/FS5700-1147045.pdf" H 8300 4100 50  0001 C CNN
+	3    8300 4100
 	1    0    0    -1
 $EndComp
-Text HLabel 2900 4500 0    50   Input ~ 0
+Text HLabel 3300 3300 0    50   Input ~ 0
 3PDT_2
-Text HLabel 2900 4800 0    50   Input ~ 0
+Text HLabel 3300 3600 0    50   Input ~ 0
 3PDT_5
-Text HLabel 3600 4700 2    50   Input ~ 0
+Text HLabel 4000 3500 2    50   Input ~ 0
 3PDT_7
-Text HLabel 3600 4600 2    50   Input ~ 0
+Text HLabel 4000 3400 2    50   Input ~ 0
 3PDT_8
-Text HLabel 3600 4500 2    50   Input ~ 0
+Text HLabel 4000 3300 2    50   Input ~ 0
 3PDT_9
-Text HLabel 3600 4800 2    50   Input ~ 0
+Text HLabel 4000 3600 2    50   Input ~ 0
 3PDT_6
-Text HLabel 2900 4700 0    50   Input ~ 0
+Text HLabel 3300 3500 0    50   Input ~ 0
 3PDT_4
-Text HLabel 2900 4600 0    50   Input ~ 0
+Text HLabel 3300 3400 0    50   Input ~ 0
 3PDT_3
-Text HLabel 2900 4400 0    50   Input ~ 0
+Text HLabel 3300 3200 0    50   Input ~ 0
 3PDT_1
 Wire Wire Line
-	2900 4500 3000 4500
+	3300 3300 3400 3300
 Wire Wire Line
-	3000 4800 2900 4800
+	3400 3600 3300 3600
 Wire Wire Line
-	3600 4600 3500 4600
+	4000 3400 3900 3400
 Wire Wire Line
-	3500 4500 3600 4500
+	3900 3300 4000 3300
 Wire Wire Line
-	3600 4700 3500 4700
+	4000 3500 3900 3500
 Wire Wire Line
-	3500 4800 3600 4800
+	3900 3600 4000 3600
 Wire Wire Line
-	2900 4700 3000 4700
+	3300 3500 3400 3500
 Wire Wire Line
-	3000 4600 2900 4600
+	3400 3400 3300 3400
 Wire Wire Line
-	2900 4400 3000 4400
+	3300 3200 3400 3200
 Wire Wire Line
-	4800 4400 4150 4400
+	5200 3200 4550 3200
 Wire Wire Line
-	4800 4500 4150 4500
+	5200 3300 4550 3300
 Wire Wire Line
-	4800 4600 4150 4600
+	5200 3400 4550 3400
 Wire Wire Line
-	4800 4700 4150 4700
+	5200 3500 4550 3500
 Wire Wire Line
-	4800 4800 4150 4800
+	5200 3600 4550 3600
 Wire Wire Line
-	5300 4800 5800 4800
+	5700 3600 6200 3600
 Wire Wire Line
-	5300 4700 5800 4700
+	5700 3500 6200 3500
 Wire Wire Line
-	5300 4600 5800 4600
+	5700 3400 6200 3400
 Wire Wire Line
-	5300 4500 5800 4500
+	5700 3300 6200 3300
 Wire Wire Line
-	6450 2950 6150 2950
+	8100 2900 7800 2900
 Wire Wire Line
-	6450 3550 6150 3550
+	8100 3500 7800 3500
 Wire Wire Line
-	6450 4150 6150 4150
+	8100 4100 7800 4100
 Wire Wire Line
-	6850 4250 7150 4250
+	8500 4200 8800 4200
 Wire Wire Line
-	6850 4050 7150 4050
+	8500 4000 8800 4000
 Wire Wire Line
-	6850 3650 7150 3650
+	8500 3600 8800 3600
 Wire Wire Line
-	6850 3450 7150 3450
+	8500 3400 8800 3400
 Wire Wire Line
-	6850 3050 7150 3050
+	8500 3000 8800 3000
 Wire Wire Line
-	6850 2850 7150 2850
-Text Label 4150 4400 0    50   ~ 0
+	8500 2800 8800 2800
+Text Label 4550 3200 0    50   ~ 0
 3PDT_1_INT
-Text Label 4150 4500 0    50   ~ 0
+Text Label 4550 3300 0    50   ~ 0
 3PDT_2_INT
-Text Label 4150 4600 0    50   ~ 0
+Text Label 4550 3400 0    50   ~ 0
 3PDT_3_INT
-Text Label 4150 4700 0    50   ~ 0
+Text Label 4550 3500 0    50   ~ 0
 3PDT_4_INT
-Text Label 4150 4800 0    50   ~ 0
+Text Label 4550 3600 0    50   ~ 0
 3PDT_5_INT
-Text Label 5800 4800 2    50   ~ 0
+Text Label 6200 3600 2    50   ~ 0
 3PDT_6_INT
-Text Label 5800 4700 2    50   ~ 0
+Text Label 6200 3500 2    50   ~ 0
 3PDT_7_INT
-Text Label 5800 4600 2    50   ~ 0
+Text Label 6200 3400 2    50   ~ 0
 3PDT_8_INT
-Text Label 5800 4500 2    50   ~ 0
+Text Label 6200 3300 2    50   ~ 0
 3PDT_9_INT
-Text Label 6150 2950 2    50   ~ 0
+Text Label 7800 2900 2    50   ~ 0
 3PDT_2_INT
-Text Label 6150 3550 2    50   ~ 0
+Text Label 7800 3500 2    50   ~ 0
 3PDT_5_INT
-Text Label 6150 4150 2    50   ~ 0
+Text Label 7800 4100 2    50   ~ 0
 3PDT_8_INT
-Text Label 7150 2850 0    50   ~ 0
+Text Label 8800 2800 0    50   ~ 0
 3PDT_1_INT
-Text Label 7150 3050 0    50   ~ 0
+Text Label 8800 3000 0    50   ~ 0
 3PDT_3_INT
-Text Label 7150 3450 0    50   ~ 0
+Text Label 8800 3400 0    50   ~ 0
 3PDT_4_INT
-Text Label 7150 3650 0    50   ~ 0
+Text Label 8800 3600 0    50   ~ 0
 3PDT_6_INT
-Text Label 7150 4050 0    50   ~ 0
+Text Label 8800 4000 0    50   ~ 0
 3PDT_7_INT
-Text Label 7150 4250 0    50   ~ 0
+Text Label 8800 4200 0    50   ~ 0
 3PDT_9_INT
 $Comp
 L Connector_Generic:Conn_02x05_Counter_Clockwise J_MAINTOAUX1
 U 1 1 5BE5C9F1
-P 3200 4600
-F 0 "J_MAINTOAUX1" H 3250 4925 50  0000 C CNN
-F 1 "Conn_02x05_Counter_Clockwise" H 3250 4926 50  0001 C CNN
-F 2 "CustomHeaders:IDCHeader_02x05_P2.54mm_Vertical_Counter_Clockwise" H 3200 4600 50  0001 C CNN
-F 3 "~" H 3200 4600 50  0001 C CNN
-	1    3200 4600
+P 3600 3400
+F 0 "J_MAINTOAUX1" H 3650 3725 50  0000 C CNN
+F 1 "Conn_02x05_Counter_Clockwise" H 3650 3726 50  0001 C CNN
+F 2 "CustomHeaders:IDCHeader_02x05_P2.54mm_Vertical_Counter_Clockwise" H 3600 3400 50  0001 C CNN
+F 3 "~" H 3600 3400 50  0001 C CNN
+	1    3600 3400
 	1    0    0    -1
 $EndComp
@@
 L Connector_Generic:Conn_02x05_Counter_Clockwise J_AUXTOMAIN1
 U 1 1 5BE5CA85
-P 5000 4600
-F 0 "J_AUXTOMAIN1" H 5050 4925 50  0000 C CNN
-F 1 "Conn_02x05_Counter_Clockwise" H 5050 4926 50  0001 C CNN
-F 2 "CustomHeaders:IDCHeader_02x05_P2.54mm_Vertical_Counter_Clockwise" H 5000 4600 50  0001 C CNN
-F 3 "~" H 5000 4600 50  0001 C CNN
-	1    5000 4600
+P 5400 3400
+F 0 "J_AUXTOMAIN1" H 5450 3725 50  0000 C CNN
+F 1 "Conn_02x05_Counter_Clockwise" H 5450 3726 50  0001 C CNN
+F 2 "CustomHeaders:IDCHeader_02x05_P2.54mm_Vertical_Counter_Clockwise" H 5400 3400 50  0001 C CNN
+F 3 "~" H 5400 3400 50  0001 C CNN
+	1    5400 3400
 	1    0    0    -1
 $EndComp

Commit message: Final RevA
Parts:
- J_MAINTOAUX1: footprint CustomHeaders:IDCHeader_02x05_P2.54mm_Vertical_Counter_Clockwise -> CustomHeaders:IDCHeader_02x05_P2.54mm_Vertical_Clockwise
- SW_EN1: Mfr. No: (none) -> FS57003PLT2B2M2QE; Mfr: (none) -> E-Switch; MouserNo (none) -> 612-FS573PLT2B2M2QE; Type (none) -> 3PDT ON-ON LATCHING
- SW_EN1: Mfr. No: (none) -> FS573PLT2B2M2QE; Mfr: (none) -> E-Switch; MouserNo (none) -> 612-FS573PLT2B2M2QE; Type (none) -> 3PDT ON-ON LATCHING
Changed lines of the file:
@@
 F 2 "custom_sw:SW_3PDT_W18MM_L17.3MM_P5.3MM_D2MM" H 8300 2900 50  0001 C CNN
 F 3 "https://www.mouser.co.uk/datasheet/2/140/FS5700-1147045.pdf" H 8300 2900 50  0001 C CNN
+F 4 "612-FS573PLT2B2M2QE" H 8300 2900 50  0001 C CNN "MouserNo"
+F 5 "FS57003PLT2B2M2QE" H 8300 2900 50  0001 C CNN "Mfr. No:"
+F 6 "E-Switch" H 8300 2900 50  0001 C CNN "Mfr:"
+F 7 "3PDT ON-ON LATCHING" H 8300 2900 50  0001 C CNN "Type"
 	1    8300 2900
 	1    0    0    -1
@@
 F 2 "custom_sw:SW_3PDT_W18MM_L17.3MM_P5.3MM_D2MM" H 8300 3500 50  0001 C CNN
 F 3 "https://www.mouser.co.uk/datasheet/2/140/FS5700-1147045.pdf" H 8300 3500 50  0001 C CNN
+F 4 "612-FS573PLT2B2M2QE" H 8300 3500 50  0001 C CNN "MouserNo"
+F 5 "FS573PLT2B2M2QE" H 8300 3500 50  0001 C CNN "Mfr. No:"
+F 6 "E-Switch" H 8300 3500 50  0001 C CNN "Mfr:"
+F 7 "3PDT ON-ON LATCHING" H 8300 3500 50  0001 C CNN "Type"
 	2    8300 3500
 	1    0    0    -1
@@
 F 2 "custom_sw:SW_3PDT_W18MM_L17.3MM_P5.3MM_D2MM" H 8300 4100 50  0001 C CNN
 F 3 "https://www.mouser.co.uk/datasheet/2/140/FS5700-1147045.pdf" H 8300 4100 50  0001 C CNN
+F 4 "612-FS573PLT2B2M2QE" H 8300 4100 50  0001 C CNN "MouserNo"
+F 5 "FS573PLT2B2M2QE" H 8300 4100 50  0001 C CNN "Mfr. No:"
+F 6 "E-Switch" H 8300 4100 50  0001 C CNN "Mfr:"
+F 7 "3PDT ON-ON LATCHING" H 8300 4100 50  0001 C CNN "Type"
 	3    8300 4100
 	1    0    0    -1
@@
 F 0 "J_MAINTOAUX1" H 3650 3725 50  0000 C CNN
 F 1 "Conn_02x05_Counter_Clockwise" H 3650 3726 50  0001 C CNN
-F 2 "CustomHeaders:IDCHeader_02x05_P2.54mm_Vertical_Counter_Clockwise" H 3600 3400 50  0001 C CNN
+F 2 "CustomHeaders:IDCHeader_02x05_P2.54mm_Vertical_Clockwise" H 3600 3400 50  0001 C CNN
 F 3 "~" H 3600 3400 50  0001 C CNN
 	1    3600 3400

Commit message: Added second 555 IC bypass cap
Connections:
- no-connect marks 0 -> 2
Changed lines of the file:
@@
 	1    0    0    -1
 $EndComp
+NoConn ~ 3900 3200
+NoConn ~ 5700 3200
 $EndSCHEMATC
