File: 555PWMTremolo/555PWMTremolo_Clock.sch (KiCad schematic (older format))
At the start: 14 parts

Commit message: Completed 555PWMTremolo Layout RevA
Parts:
- C_BP1: footprint (none) -> Capacitor_SMD:C_0805_2012Metric_Pad1.15x1.40mm_HandSolder
- P_OSCOFF1, P_OSCON1: footprint Potentiometer_THT:Potentiometer_Alps_RK09K_Single_Vertical -> Potentiometer_THT:Potentiometer_Alps_RK09L_Single_Vertical
Connections:
- wire segments 58 -> 59
Changed lines of the file:
@@
 F 0 "P_OSCON1" H 2850 3900 50  0000 C CNN
 F 1 "B10K" H 2850 4000 50  0000 C CNN
-F 2 "Potentiometer_THT:Potentiometer_Alps_RK09K_Single_Vertical" H 2400 3950 50  0001 C CNN
+F 2 "Potentiometer_THT:Potentiometer_Alps_RK09L_Single_Vertical" H 2400 3950 50  0001 C CNN
 F 3 "~" H 2400 3950 50  0001 C CNN
 	1    2400 3950
@@
 F 0 "P_OSCOFF1" H 2900 3300 50  0000 C CNN
 F 1 "B10K" H 2800 3200 50  0000 C CNN
-F 2 "Potentiometer_THT:Potentiometer_Alps_RK09K_Single_Vertical" H 2400 3150 50  0001 C CNN
+F 2 "Potentiometer_THT:Potentiometer_Alps_RK09L_Single_Vertical" H 2400 3150 50  0001 C CNN
 F 3 "~" H 2400 3150 50  0001 C CNN
 	1    2400 3150
@@
 Connection ~ 4000 2200
 Wire Wire Line
-	4000 2200 4000 2750
+	4000 2200 4000 2500
 Wire Wire Line
 	2400 2200 2400 2500
@@
 F 0 "C_BP1" H 5215 2695 50  0000 L CNN
 F 1 "100nF" H 5215 2606 50  0000 L CNN
-F 2 "" H 5138 2500 50  0001 C CNN
+F 2 "Capacitor_SMD:C_0805_2012Metric_Pad1.15x1.40mm_HandSolder" H 5138 2500 50  0001 C CNN
 F 3 "~" H 5100 2650 50  0001 C CNN
 	1    5100 2650
@@
 Text HLabel 5100 3200 3    50   Input ~ 0
 GND
+$Comp
+L power:PWR_FLAG #FLG0103
+U 1 1 5BE575F8
+P 4000 2500
+F 0 "#FLG0103" H 4000 2575 50  0001 C CNN
+F 1 "PWR_FLAG" V 4000 2627 50  0000 L CNN
+F 2 "" H 4000 2500 50  0001 C CNN
+F 3 "~" H 4000 2500 50  0001 C CNN
+	1    4000 2500
+	0    1    1    0
+$EndComp
+Connection ~ 4000 2500
+Wire Wire Line
+	4000 2500 4000 2750
 $EndSCHEMATC

Commit message: Tidied up 555 layout
Parts:
- removed U_OPTO1: 4N35, Package_DIP:SMDIP-6_W7.62mm, symbol Isolator:4N35
- added U_OPTO1: LTV-357T, Package_SO:SO-4_4.4x2.3mm_P1.27mm, symbol Isolator:LTV-357T
Connections:
- no-connect marks 1 -> 0
Changed lines of the file:
@@
 $EndDescr
-$Comp
-L Isolator:4N35 U_OPTO1
-U 1 1 5BF61C95
-P 8700 2800
-F 0 "U_OPTO1" V 8750 3350 50  0000 R CNN
-F 1 "4N35" V 8650 3300 50  0000 R CNN
-F 2 "Package_DIP:SMDIP-6_W7.62mm" H 8500 2600 50  0001 L CIN
-F 3 "https://www.vishay.com/docs/81181/4n35.pdf" H 8700 2800 50  0001 L CNN
-	1    8700 2800
-	0    -1   -1   0
-$EndComp
 $Comp
 L Device:LED D_LED1
@@
 Wire Wire Line
 	8800 2400 9100 2400
-NoConn ~ 8600 2500
 $Comp
 L Device:R R_LPF1
@@
 CLK_OUT
 Wire Wire Line
-	8700 2100 8700 2500
-Wire Wire Line
-	8700 2100 9650 2100
+	8600 2100 8600 2500
+Wire Wire Line
+	8600 2100 9650 2100
 Text HLabel 9100 4300 3    50   Input ~ 0
 GND
@@
 Wire Wire Line
 	4000 2500 4000 2750
+$Comp
+L Isolator:LTV-357T U_OPTO1
+U 1 1 5BE5F080
+P 8700 2800
+F 0 "U_OPTO1" V 8750 3350 50  0000 R CNN
+F 1 "LTV-357T" V 8650 3350 50  0000 R CNN
+F 2 "Package_SO:SO-4_4.4x2.3mm_P1.27mm" H 8500 2600 50  0001 L CIN
+F 3 "https://www.buerklin.com/medias/sys_master/download/download/h91/ha0/8892020588574.pdf" H 8700 2800 50  0001 L CNN
+	1    8700 2800
+	0    -1   -1   0
+$EndComp
 $EndSCHEMATC

Commit message: Final RevA
Parts:
- added CP_SLOW1: 220uF, Capacitor_SMD:CP_Elec_6.3x5.4, symbol Device:CP
- added R_OSCLIMIT1: 100R, Resistor_SMD:R_0805_2012Metric_Pad1.15x1.40mm_HandSolder, symbol Device:R
- added SW_ATTACK1: SW_SPDT, DailywellSwitches:Dailywell_SPDT, symbol Switch:SW_SPDT
- renumbered CP_LPF1 to CP_FAST1
Connections:
- wire segments 59 -> 62
Changed lines of the file:
@@
 L Device:LED D_LED1
 U 1 1 5BF61C9C
-P 7200 3400
-F 0 "D_LED1" H 7200 3150 50  0000 C CNN
-F 1 "LED" H 7200 3250 50  0000 C CNN
-F 2 "LED_THT:LED_D5.0mm" H 7200 3400 50  0001 C CNN
-F 3 "~" H 7200 3400 50  0001 C CNN
-	1    7200 3400
+P 6600 3400
+F 0 "D_LED1" H 6600 3150 50  0000 C CNN
+F 1 "LED" H 6600 3250 50  0000 C CNN
+F 2 "LED_THT:LED_D5.0mm" H 6600 3400 50  0001 C CNN
+F 3 "~" H 6600 3400 50  0001 C CNN
+	1    6600 3400
 	-1   0    0    1
 $EndComp
@@
 	8600 3400 8600 3100
 Wire Wire Line
-	9100 3400 9100 4300
+	9600 3400 9600 4300
 Wire Wire Line
 	8800 2500 8800 2400
 Wire Wire Line
-	8800 2400 9100 2400
+	8800 2400 9600 2400
 $Comp
 L Device:R R_LPF1
 U 1 1 5BF61CAE
-P 6600 3400
-F 0 "R_LPF1" V 6350 3400 50  0000 C CNN
-F 1 "100R" V 6450 3400 50  0000 C CNN
-F 2 "Resistor_SMD:R_0805_2012Metric_Pad1.15x1.40mm_HandSolder" V 6530 3400 50  0001 C CNN
-F 3 "~" H 6600 3400 50  0001 C CNN
-	1    6600 3400
+P 6000 3400
+F 0 "R_LPF1" V 5750 3400 50  0000 C CNN
+F 1 "100R" V 5850 3400 50  0000 C CNN
+F 2 "Resistor_SMD:R_0805_2012Metric_Pad1.15x1.40mm_HandSolder" V 5930 3400 50  0001 C CNN
+F 3 "~" H 6000 3400 50  0001 C CNN
+	1    6000 3400
 	0    1    1    0
 $EndComp
 $Comp
-L Device:CP CP_LPF1
+L Device:CP CP_FAST1
 U 1 1 5BF61CB5
-P 8600 3850
-F 0 "CP_LPF1" H 8717 3895 50  0000 L CNN
-F 1 "22uF" H 8717 3806 50  0000 L CNN
-F 2 "Capacitor_SMD:CP_Elec_4x5.4" H 8638 3700 50  0001 C CNN
-F 3 "~" H 8600 3850 50  0001 C CNN
-	1    8600 3850
-	1    0    0    -1
-$EndComp
-Wire Wire Line
-	8600 3400 8600 3700
-Wire Wire Line
-	8600 3400 7700 3400
-Connection ~ 8600 3400
-Wire Wire Line
-	6750 3400 6900 3400
+P 8900 4450
+F 0 "CP_FAST1" H 9017 4495 50  0000 L CNN
+F 1 "22uF" H 9017 4406 50  0000 L CNN
+F 2 "Capacitor_SMD:CP_Elec_4x5.4" H 8938 4300 50  0001 C CNN
+F 3 "~" H 8900 4450 50  0001 C CNN
+	1    8900 4450
+	1    0    0    -1
+$EndComp
+Wire Wire Line
+	8700 4000 8900 4300
+Wire Wire Line
+	8600 3400 7100 3400
+Wire Wire Line
+	6150 3400 6300 3400
 Wire Wire Line
 	8800 3100 8800 3400
 Wire Wire Line
-	8800 3400 9100 3400
-Wire Wire Line
-	9100 2400 9100 3400
-Connection ~ 9100 3400
+	8800 3400 9600 3400
+Wire Wire Line
+	9600 2400 9600 3400
+Connection ~ 9600 3400
 Text HLabel 9650 2100 2    50   Input ~ 0
 CLK_OUT
@@
 Wire Wire Line
 	8600 2100 9650 2100
-Text HLabel 9100 4300 3    50   Input ~ 0
-GND
-Wire Wire Line
-	8600 4000 8600 4300
-Text HLabel 8600 4300 3    50   Input ~ 0
+Text HLabel 9600 4300 3    50   Input ~ 0
+GND
+Text HLabel 8900 4900 3    50   Input ~ 0
 GND
 $Comp
 L Device:C C_LPFOPT2
 U 1 1 5C18730A
-P 7700 3850
-F 0 "C_LPFOPT2" H 7815 3896 50  0000 L CNN
-F 1 "10uF" H 7815 3805 50  0000 L CNN
-F 2 "Capacitor_SMD:C_0805_2012Metric_Pad1.15x1.40mm_HandSolder" H 7738 3700 50  0001 C CNN
-F 3 "~" H 7700 3850 50  0001 C CNN
-	1    7700 3850
+P 7100 3850
+F 0 "C_LPFOPT2" H 7215 3896 50  0000 L CNN
+F 1 "10uF" H 7215 3805 50  0000 L CNN
+F 2 "Capacitor_SMD:C_0805_2012Metric_Pad1.15x1.40mm_HandSolder" H 7138 3700 50  0001 C CNN
+F 3 "~" H 7100 3850 50  0001 C CNN
+	1    7100 3850
 	1    0    0    -1
 $EndComp
@@
 L Device:C C_LPFOPT1
 U 1 1 5C18735B
-P 6900 3850
-F 0 "C_LPFOPT1" H 7015 3896 50  0000 L CNN
-F 1 "100nF" H 7015 3805 50  0000 L CNN
-F 2 "Capacitor_SMD:C_0805_2012Metric_Pad1.15x1.40mm_HandSolder" H 6938 3700 50  0001 C CNN
-F 3 "~" H 6900 3850 50  0001 C CNN
-	1    6900 3850
-	1    0    0    -1
-$EndComp
-Wire Wire Line
-	6900 3700 6900 3400
-Connection ~ 6900 3400
-Wire Wire Line
-	6900 3400 7050 3400
-Wire Wire Line
-	7700 3700 7700 3400
-Connection ~ 7700 3400
-Wire Wire Line
-	7700 3400 7350 3400
-Wire Wire Line
-	7700 4000 7700 4300
-Text HLabel 7700 4300 3    50   Input ~ 0
-GND
-Wire Wire Line
-	6900 4000 6900 4300
-Text HLabel 6900 4300 3    50   Input ~ 0
+P 6300 3850
+F 0 "C_LPFOPT1" H 6415 3896 50  0000 L CNN
+F 1 "100nF" H 6415 3805 50  0000 L CNN
+F 2 "Capacitor_SMD:C_0805_2012Metric_Pad1.15x1.40mm_HandSolder" H 6338 3700 50  0001 C CNN
+F 3 "~" H 6300 3850 50  0001 C CNN
+	1    6300 3850
+	1    0    0    -1
+$EndComp
+Wire Wire Line
+	6300 3700 6300 3400
+Connection ~ 6300 3400
+Wire Wire Line
+	6300 3400 6450 3400
+Wire Wire Line
+	7100 3700 7100 3400
+Connection ~ 7100 3400
+Wire Wire Line
+	7100 3400 6750 3400
+Wire Wire Line
+	7100 4000 7100 4300
+Text HLabel 7100 4300 3    50   Input ~ 0
+GND
+Wire Wire Line
+	6300 4000 6300 4300
+Text HLabel 6300 4300 3    50   Input ~ 0
 GND
 Text HLabel 2400 5800 3    50   Input ~ 0
@@
 	5750 3800 5750 3400
 Wire Wire Line
-	5750 3400 6450 3400
+	5750 3400 5850 3400
 Wire Wire Line
 	4500 3900 4700 3900
@@
 	3500 3600 2400 3600
 Wire Wire Line
-	4000 1950 4000 2200
-Wire Wire Line
 	2400 2200 4000 2200
 Connection ~ 4000 2200
 Wire Wire Line
-	4000 2200 4000 2500
-Wire Wire Line
 	2400 2200 2400 2500
 Wire Wire Line
@@
 	2400 4600 2400 4900
 Connection ~ 2400 4900
-Text HLabel 4000 1950 1    50   Input ~ 0
+Text HLabel 4000 1500 1    50   Input ~ 0
 VCC
 $Comp
@@
 Text HLabel 5100 3200 3    50   Input ~ 0
 GND
-$Comp
-L power:PWR_FLAG #FLG0103
-U 1 1 5BE575F8
-P 4000 2500
-F 0 "#FLG0103" H 4000 2575 50  0001 C CNN
-F 1 "PWR_FLAG" V 4000 2627 50  0000 L CNN
-F 2 "" H 4000 2500 50  0001 C CNN
-F 3 "~" H 4000 2500 50  0001 C CNN
-	1    4000 2500
-	0    1    1    0
-$EndComp
-Connection ~ 4000 2500
-Wire Wire Line
-	4000 2500 4000 2750
 $Comp
 L Isolator:LTV-357T U_OPTO1
@@
 	0    -1   -1   0
 $EndComp
+$Comp
+L Device:R R_OSCLIMIT1
+U 1 1 5BE63342
+P 4000 1850
+F 0 "R_OSCLIMIT1" H 4070 1896 50  0000 L CNN
+F 1 "100R" H 4070 1805 50  0000 L CNN
+F 2 "Resistor_SMD:R_0805_2012Metric_Pad1.15x1.40mm_HandSolder" V 3930 1850 50  0001 C CNN
+F 3 "~" H 4000 1850 50  0001 C CNN
+	1    4000 1850
+	1    0    0    -1
+$EndComp
+Wire Wire Line
+	4000 1500 4000 1700
+Wire Wire Line
+	4000 2000 4000 2200
+Wire Wire Line
+	4000 2200 4000 2750
+$Comp
+L Switch:SW_SPDT SW_ATTACK1
+U 1 1 5BE6888F
+P 8600 3800
+F 0 "SW_ATTACK1" V 8600 3948 50  0000 L CNN
+F 1 "SW_SPDT" V 8645 3948 50  0001 L CNN
+F 2 "DailywellSwitches:Dailywell_SPDT" H 8600 3800 50  0001 C CNN
+F 3 "" H 8600 3800 50  0001 C CNN
+	1    8600 3800
+	0    1    1    0
+$EndComp
+Wire Wire Line
+	8900 4600 8900 4900
+Wire Wire Line
+	8600 3600 8600 3400
+Connection ~ 8600 3400
+$Comp
+L Device:CP CP_SLOW1
+U 1 1 5BE6F69D
+P 8300 4450
+F 0 "CP_SLOW1" H 7800 4500 50  0000 L CNN
+F 1 "220uF" H 7850 4350 50  0000 L CNN
+F 2 "Capacitor_SMD:CP_Elec_6.3x5.4" H 8338 4300 50  0001 C CNN
+F 3 "~" H 8300 4450 50  0001 C CNN
+	1    8300 4450
+	1    0    0    -1
+$EndComp
+Wire Wire Line
+	8300 4300 8500 4000
+Text HLabel 8300 4900 3    50   Input ~ 0
+GND
+Wire Wire Line
+	8300 4600 8300 4900
 $EndSCHEMATC

Commit message: Final RevA
Parts:
- CP_FAST1: Diameter (none) -> 4mm; ESR (none) -> 45mOhms; Mfr. No: (none) -> 875105240003; Mfr: (none) -> Wurth; MouserNo (none) -> 710-875105240003; Tolerance (none) -> 20%; Type (none) -> Aluminium Organic Polymer Capacitors WCAP-PSLP 10V 22uF 20%; Voltage Rating DC (none) -> 10 DC
- CP_SLOW1: Diameter (none) -> 6 mm; ESR (none) -> 160 mOhms; Mfr. No: (none) -> EEE-FPC221XAP; Mfr: (none) -> Panasonic; MouserNo (none) -> 667-EEE-FPC221XAP; Tolerance (none) -> 20 %; Type (none) -> Aluminium Electrolytic Capacitors - SMD; Voltage Rating DC (none) -> 16 VDC
- P_OSCOFF1, P_OSCON1: Mfr. No: (none) -> RK09L1140A66; Mfr: (none) -> ALPS; MouserNo (none) -> 688-RK09L1140A66; Type (none) -> 1GANG LINEAR 20% FLATTED 1TURN
- R_OSCLIMIT1: Mfr. No: (none) -> CRS0805AFX1000LF; Mfr: (none) -> Bourns; MouserNo (none) -> 652-CRS0805AFX1000LF; Type (none) -> Thick Film Resistors - SMD 100 ohm 1% 1/4W TC100
- SW_ATTACK1: Mfr. No: (none) -> 108-2MS1T1B1M2QE-EVX; Mfr: (none) -> Mountain Switch; MouserNo (none) -> 108-2MS1T1B1M2QE-EVX; Type (none) -> TOGGLE SPDT ON-ON PC MOUNT
- U_OPTO1: Mfr. No: (none) -> ACPL-217-50BE; Mfr: (none) -> Broadcom / Avago; MouserNo (none) -> 630-ACPL-217-50BE; Type (none) -> Transistor Output Optocouplers 3000Vrms 50% CTR
- U_OSC1: Mfr. No: (none) -> TLC555CDR; Mfr: (none) -> Texas Instruments; MouserNo (none) -> 595-TLC555CDR; Type (none) -> LinCMOS Clock & Timer IC
Changed lines of the file:
@@
 F 1 "22uF" H 9017 4406 50  0000 L CNN
 F 2 "Capacitor_SMD:CP_Elec_4x5.4" H 8938 4300 50  0001 C CNN
-F 3 "~" H 8900 4450 50  0001 C CNN
+F 3 "https://www.mouser.co.uk/datasheet/2/445/875105240003-540627.pdf" H 8900 4450 50  0001 C CNN
+F 4 "710-875105240003" H 8900 4450 50  0001 C CNN "MouserNo"
+F 5 "875105240003" H 8900 4450 50  0001 C CNN "Mfr. No:"
+F 6 "Wurth" H 8900 4450 50  0001 C CNN "Mfr:"
+F 7 "Aluminium Organic Polymer Capacitors WCAP-PSLP 10V 22uF 20%" H 8900 4450 50  0001 C CNN "Type"
+F 8 "45mOhms" H 8900 4450 50  0001 C CNN "ESR"
+F 9 "20%" H 8900 4450 50  0001 C CNN "Tolerance"
+F 10 "10 DC" H 8900 4450 50  0001 C CNN "Voltage Rating DC"
+F 11 "4mm" H 8900 4450 50  0001 C CNN "Diameter"
 	1    8900 4450
 	1    0    0    -1
@@
 F 1 "B10K" H 2850 4000 50  0000 C CNN
 F 2 "Potentiometer_THT:Potentiometer_Alps_RK09L_Single_Vertical" H 2400 3950 50  0001 C CNN
-F 3 "~" H 2400 3950 50  0001 C CNN
+F 3 "https://www.mouser.co.uk/datasheet/2/15/RK09L-1370814.pdf" H 2400 3950 50  0001 C CNN
+F 4 "688-RK09L1140A66" H 2400 3950 50  0001 C CNN "MouserNo"
+F 5 "RK09L1140A66" H 2400 3950 50  0001 C CNN "Mfr. No:"
+F 6 "ALPS" H 2400 3950 50  0001 C CNN "Mfr:"
+F 7 "1GANG LINEAR 20% FLATTED 1TURN" H 2400 3950 50  0001 C CNN "Type"
 	1    2400 3950
 	-1   0    0    1
@@
 F 1 "TLC555" H 4250 4350 50  0000 C CNN
 F 2 "Package_SO:SOIC-8_3.9x4.9mm_P1.27mm" H 4050 3550 50  0001 L CNN
-F 3 "http://www.ti.com/lit/ds/symlink/tlc555.pdf" H 4650 3250 50  0001 C CNN
+F 3 "http://www.ti.com/general/docs/suppproductinfo.tsp?distId=26&gotoUrl=http%3A%2F%2Fwww.ti.com%2Flit%2Fgpn%2Ftlc555" H 4650 3250 50  0001 C CNN
+F 4 "595-TLC555CDR" H 4000 3800 50  0001 C CNN "MouserNo"
+F 5 "TLC555CDR" H 4000 3800 50  0001 C CNN "Mfr. No:"
+F 6 "Texas Instruments" H 4000 3800 50  0001 C CNN "Mfr:"
+F 7 "LinCMOS Clock & Timer IC" H 4000 3800 50  0001 C CNN "Type"
 	1    4000 3800
 	1    0    0    -1
@@
 F 1 "B10K" H 2800 3200 50  0000 C CNN
 F 2 "Potentiometer_THT:Potentiometer_Alps_RK09L_Single_Vertical" H 2400 3150 50  0001 C CNN
-F 3 "~" H 2400 3150 50  0001 C CNN
+F 3 "https://www.mouser.co.uk/datasheet/2/15/RK09L-1370814.pdf" H 2400 3150 50  0001 C CNN
+F 4 "688-RK09L1140A66" H 2400 3150 50  0001 C CNN "MouserNo"
+F 5 "RK09L1140A66" H 2400 3150 50  0001 C CNN "Mfr. No:"
+F 6 "ALPS" H 2400 3150 50  0001 C CNN "Mfr:"
+F 7 "1GANG LINEAR 20% FLATTED 1TURN" H 2400 3150 50  0001 C CNN "Type"
 	1    2400 3150
 	-1   0    0    -1
@@
 F 1 "LTV-357T" V 8650 3350 50  0000 R CNN
 F 2 "Package_SO:SO-4_4.4x2.3mm_P1.27mm" H 8500 2600 50  0001 L CIN
-F 3 "https://www.buerklin.com/medias/sys_master/download/download/h91/ha0/8892020588574.pdf" H 8700 2800 50  0001 L CNN
+F 3 "https://docs.broadcom.com/docs/av02-0470en" H 8700 2800 50  0001 L CNN
+F 4 "630-ACPL-217-50BE" H 8700 2800 50  0001 C CNN "MouserNo"
+F 5 "ACPL-217-50BE" H 8700 2800 50  0001 C CNN "Mfr. No:"
+F 6 "Broadcom / Avago" H 8700 2800 50  0001 C CNN "Mfr:"
+F 7 "Transistor Output Optocouplers 3000Vrms 50% CTR" H 8700 2800 50  0001 C CNN "Type"
 	1    8700 2800
 	0    -1   -1   0
@@
 F 1 "100R" H 4070 1805 50  0000 L CNN
 F 2 "Resistor_SMD:R_0805_2012Metric_Pad1.15x1.40mm_HandSolder" V 3930 1850 50  0001 C CNN
-F 3 "~" H 4000 1850 50  0001 C CNN
+F 3 "https://www.mouser.co.uk/datasheet/2/54/rs-a-1222350.pdf" H 4000 1850 50  0001 C CNN
+F 4 "652-CRS0805AFX1000LF" H 4000 1850 50  0001 C CNN "MouserNo"
+F 5 "CRS0805AFX1000LF" H 4000 1850 50  0001 C CNN "Mfr. No:"
+F 6 "Bourns" H 4000 1850 50  0001 C CNN "Mfr:"
+F 7 "Thick Film Resistors - SMD 100 ohm 1% 1/4W TC100" H 4000 1850 50  0001 C CNN "Type"
 	1    4000 1850
 	1    0    0    -1
@@
 F 1 "SW_SPDT" V 8645 3948 50  0001 L CNN
 F 2 "DailywellSwitches:Dailywell_SPDT" H 8600 3800 50  0001 C CNN
-F 3 "" H 8600 3800 50  0001 C CNN
+F 3 "https://www.mouser.co.uk/datasheet/2/209/MS-100786-1172382.pdf" H 8600 3800 50  0001 C CNN
+F 4 "108-2MS1T1B1M2QE-EVX" H 8600 3800 50  0001 C CNN "MouserNo"
+F 5 "108-2MS1T1B1M2QE-EVX" H 8600 3800 50  0001 C CNN "Mfr. No:"
+F 6 "Mountain Switch" H 8600 3800 50  0001 C CNN "Mfr:"
+F 7 "TOGGLE SPDT ON-ON PC MOUNT" H 8600 3800 50  0001 C CNN "Type"
 	1    8600 3800
 	0    1    1    0
@@
 F 1 "220uF" H 7850 4350 50  0000 L CNN
 F 2 "Capacitor_SMD:CP_Elec_6.3x5.4" H 8338 4300 50  0001 C CNN
-F 3 "~" H 8300 4450 50  0001 C CNN
+F 3 "https://www.mouser.co.uk/datasheet/2/315/ABA0000C1184-947404.pdf" H 8300 4450 50  0001 C CNN
+F 4 "667-EEE-FPC221XAP" H 8300 4450 50  0001 C CNN "MouserNo"
+F 5 "EEE-FPC221XAP" H 8300 4450 50  0001 C CNN "Mfr. No:"
+F 6 "Panasonic" H 8300 4450 50  0001 C CNN "Mfr:"
+F 7 "Aluminium Electrolytic Capacitors - SMD  " H 8300 4450 50  0001 C CNN "Type"
+F 8 "6 mm" H 8300 4450 50  0001 C CNN "Diameter"
+F 9 "160 mOhms" H 8300 4450 50  0001 C CNN "ESR"
+F 10 "16 VDC" H 8300 4450 50  0001 C CNN "Voltage Rating DC"
+F 11 "20 %" H 8300 4450 50  0001 C CNN "Tolerance"
 	1    8300 4450
 	1    0    0    -1

Commit message: Added second 555 IC bypass cap
Parts:
- added C_BP2: 47uF, Capacitor_SMD:C_0805_2012Metric_Pad1.15x1.40mm_HandSolder, symbol Device:C
- R_OSCLIMIT1: value 100R -> 330R
- R_OSCOFF1, R_OSCON1: value 100R -> 220R
Connections:
- wire segments 62 -> 65
Changed lines of the file:
@@
 P 2400 4450
 F 0 "R_OSCON1" H 2050 4500 50  0000 C CNN
-F 1 "100R" H 2050 4400 50  0000 C CNN
+F 1 "220R" H 2050 4400 50  0000 C CNN
 F 2 "Resistor_SMD:R_0805_2012Metric_Pad1.15x1.40mm_HandSolder" V 2330 4450 50  0001 C CNN
 F 3 "~" H 2400 4450 50  0001 C CNN
@@
 P 2400 2650
 F 0 "R_OSCOFF1" H 1900 2600 50  0000 C CNN
-F 1 "100R" H 1950 2700 50  0000 C CNN
+F 1 "220R" H 1950 2700 50  0000 C CNN
 F 2 "Resistor_SMD:R_0805_2012Metric_Pad1.15x1.40mm_HandSolder" V 2330 2650 50  0001 C CNN
 F 3 "~" H 2400 2650 50  0001 C CNN
@@
 P 4000 1850
 F 0 "R_OSCLIMIT1" H 4070 1896 50  0000 L CNN
-F 1 "100R" H 4070 1805 50  0000 L CNN
+F 1 "330R" H 4070 1805 50  0000 L CNN
 F 2 "Resistor_SMD:R_0805_2012Metric_Pad1.15x1.40mm_HandSolder" V 3930 1850 50  0001 C CNN
 F 3 "https://www.mouser.co.uk/datasheet/2/54/rs-a-1222350.pdf" H 4000 1850 50  0001 C CNN
@@
 Wire Wire Line
 	8300 4600 8300 4900
+Wire Wire Line
+	5600 2500 5600 2200
+Wire Wire Line
+	5600 2200 5100 2200
+Connection ~ 5100 2200
+Wire Wire Line
+	5600 2800 5600 3200
+Text HLabel 5600 3200 3    50   Input ~ 0
+GND
+$Comp
+L Device:C C_BP2
+U 1 1 5BEDE887
+P 5600 2650
+F 0 "C_BP2" H 5715 2696 50  0000 L CNN
+F 1 "47uF" H 5715 2605 50  0000 L CNN
+F 2 "Capacitor_SMD:C_0805_2012Metric_Pad1.15x1.40mm_HandSolder" H 5638 2500 50  0001 C CNN
+F 3 "~" H 5600 2650 50  0001 C CNN
+	1    5600 2650
+	1    0    0    -1
+$EndComp
 $EndSCHEMATC

Commit message: Added second 555 IC bypass cap
Parts:
- R_OSCOFF1, R_OSCON1: value 220R -> 1K
Other:
- note added: "(Optional)"
Changed lines of the file:
@@
 P 2400 4450
 F 0 "R_OSCON1" H 2050 4500 50  0000 C CNN
-F 1 "220R" H 2050 4400 50  0000 C CNN
+F 1 "1K" H 2050 4400 50  0000 C CNN
 F 2 "Resistor_SMD:R_0805_2012Metric_Pad1.15x1.40mm_HandSolder" V 2330 4450 50  0001 C CNN
 F 3 "~" H 2400 4450 50  0001 C CNN
@@
 P 2400 2650
 F 0 "R_OSCOFF1" H 1900 2600 50  0000 C CNN
-F 1 "220R" H 1950 2700 50  0000 C CNN
+F 1 "1K" H 1950 2700 50  0000 C CNN
 F 2 "Resistor_SMD:R_0805_2012Metric_Pad1.15x1.40mm_HandSolder" V 2330 2650 50  0001 C CNN
 F 3 "~" H 2400 2650 50  0001 C CNN
@@
 	1    0    0    -1
 $EndComp
+Text Notes 6400 4050 0    50   ~ 0
+(Optional)
+Text Notes 7200 4050 0    50   ~ 0
+(Optional)
 $EndSCHEMATC
