File: 555PWMTremolo/555PWMTremolo.sch (KiCad schematic (older format))
At the start: 20 parts

Commit message: Completed 555PWMTremolo Layout RevA
Changed lines of the file:
@@
 Wire Wire Line
 	4200 9300 4200 9950
-$Comp
-L power:GND #PWR03
-U 1 1 5BE0D7C8
-P 4200 9950
-F 0 "#PWR03" H 4200 9700 50  0001 C CNN
-F 1 "GND" H 4205 9779 50  0001 C CNN
-F 2 "" H 4200 9950 50  0001 C CNN
-F 3 "" H 4200 9950 50  0001 C CNN
-	1    4200 9950
-	1    0    0    -1
-$EndComp
 Wire Wire Line
 	3800 9000 3550 9000
 Wire Wire Line
 	3550 9000 3550 9950
-$Comp
-L power:GND #PWR02
-U 1 1 5BE0D8B2
-P 3550 9950
-F 0 "#PWR02" H 3550 9700 50  0001 C CNN
-F 1 "GND" H 3555 9779 50  0001 C CNN
-F 2 "" H 3550 9950 50  0001 C CNN
-F 3 "" H 3550 9950 50  0001 C CNN
-	1    3550 9950
-	1    0    0    -1
-$EndComp
 NoConn ~ 3800 8800
 Wire Wire Line
@@
 Wire Wire Line
 	8600 9000 8600 9450
-$Comp
-L power:GND #PWR011
-U 1 1 5BE0F8AC
-P 8600 9950
-F 0 "#PWR011" H 8600 9700 50  0001 C CNN
-F 1 "GND" H 8605 9779 50  0001 C CNN
-F 2 "" H 8600 9950 50  0001 C CNN
-F 3 "" H 8600 9950 50  0001 C CNN
-	1    8600 9950
-	1    0    0    -1
-$EndComp
 Wire Wire Line
 	6750 9000 6750 9100
-$Comp
-L power:GND #PWR08
-U 1 1 5BE0FCBF
-P 6750 9950
-F 0 "#PWR08" H 6750 9700 50  0001 C CNN
-F 1 "GND" H 6755 9779 50  0001 C CNN
-F 2 "" H 6750 9950 50  0001 C CNN
-F 3 "" H 6750 9950 50  0001 C CNN
-	1    6750 9950
-	1    0    0    -1
-$EndComp
 $Comp
 L Device:R R2
@@
 $EndComp
 Wire Wire Line
-	8600 9850 8600 9950
+	8600 9850 8600 10000
 Wire Wire Line
 	8600 9450 8600 9550
@@
 Wire Wire Line
 	5400 9000 5400 9950
-$Comp
-L power:GND #PWR05
-U 1 1 5BE19F49
-P 5400 9950
-F 0 "#PWR05" H 5400 9700 50  0001 C CNN
-F 1 "GND" H 5405 9779 50  0001 C CNN
-F 2 "" H 5400 9950 50  0001 C CNN
-F 3 "" H 5400 9950 50  0001 C CNN
-	1    5400 9950
-	1    0    0    -1
-$EndComp
 $Comp
 L Amplifier_Operational:TL072 U_BUF1
@@
 Wire Wire Line
 	9850 2400 9650 2400
-$Comp
-L power:GND #PWR014
-U 1 1 5BE2458F
-P 9650 4250
-F 0 "#PWR014" H 9650 4000 50  0001 C CNN
-F 1 "GND" H 9655 4079 50  0001 C CNN
-F 2 "" H 9650 4250 50  0001 C CNN
-F 3 "" H 9650 4250 50  0001 C CNN
-	1    9650 4250
-	1    0    0    -1
-$EndComp
 Wire Wire Line
 	10000 3100 9650 3100
@@
 Wire Wire Line
 	2250 9050 2250 9250
-$Comp
-L power:GND #PWR021
-U 1 1 5BE80CEE
-P 2250 9250
-F 0 "#PWR021" H 2250 9000 50  0001 C CNN
-F 1 "GND" H 2255 9079 50  0001 C CNN
-F 2 "" H 2250 9250 50  0001 C CNN
-F 3 "" H 2250 9250 50  0001 C CNN
-	1    2250 9250
-	1    0    0    -1
-$EndComp
 Wire Wire Line
 	9650 3100 9650 3600
@@
 	14150 8000 13950 8000
 Wire Wire Line
-	13950 8000 13950 8050
+	13950 8000 13950 8200
 Connection ~ 14150 8000
-$Comp
-L power:GND #PWR0102
-U 1 1 5BED3C4A
-P 13950 8050
-F 0 "#PWR0102" H 13950 7800 50  0001 C CNN
-F 1 "GND" H 13955 7879 50  0001 C CNN
-F 2 "" H 13950 8050 50  0001 C CNN
-F 3 "" H 13950 8050 50  0001 C CNN
-	1    13950 8050
-	1    0    0    -1
-$EndComp
 Wire Wire Line
 	14150 8000 14150 7950
@@
 Wire Wire Line
 	3300 9300 3300 9950
-$Comp
-L power:GND #PWR0103
-U 1 1 5BF2BDEC
-P 3300 9950
-F 0 "#PWR0103" H 3300 9700 50  0001 C CNN
-F 1 "GND" H 3305 9779 50  0001 C CNN
-F 2 "" H 3300 9950 50  0001 C CNN
-F 3 "" H 3300 9950 50  0001 C CNN
-	1    3300 9950
-	1    0    0    -1
-$EndComp
 Wire Wire Line
 	7550 2200 6100 2200
@@
 	12900 2500 12900 2950
 $Comp
-L power:GND #PWR0104
-U 1 1 5BE5BF67
-P 12900 2950
-F 0 "#PWR0104" H 12900 2700 50  0001 C CNN
-F 1 "GND" H 12905 2777 50  0001 C CNN
-F 2 "" H 12900 2950 50  0001 C CNN
-F 3 "" H 12900 2950 50  0001 C CNN
-	1    12900 2950
-	1    0    0    -1
-$EndComp
-$Comp
 L socket_custom:JACK__MONO_2P_NC J_IN1
 U 1 1 5BE61397
@@
 Wire Wire Line
 	3100 2300 3100 2750
-$Comp
-L power:GND #PWR0105
-U 1 1 5BE613A6
-P 3100 2750
-F 0 "#PWR0105" H 3100 2500 50  0001 C CNN
-F 1 "GND" H 3105 2577 50  0001 C CNN
-F 2 "" H 3100 2750 50  0001 C CNN
-F 3 "" H 3100 2750 50  0001 C CNN
-	1    3100 2750
-	-1   0    0    -1
-$EndComp
 Wire Wire Line
 	13200 2200 12650 2200
@@
 Wire Wire Line
 	7650 4800 7550 4800
-$Comp
-L power:GND #PWR0107
-U 1 1 5BFBD58F
-P 8500 5500
-F 0 "#PWR0107" H 8500 5250 50  0001 C CNN
-F 1 "GND" H 8505 5329 50  0001 C CNN
-F 2 "" H 8500 5500 50  0001 C CNN
-F 3 "" H 8500 5500 50  0001 C CNN
-	1    8500 5500
-	1    0    0    -1
-$EndComp
 Wire Wire Line
 	8500 5500 8500 5050
@@
 Wire Wire Line
 	3700 5400 3700 5750
+Text Label 3100 2750 1    50   ~ 0
+GND
+Text Label 8500 5500 1    50   ~ 0
+GND
+Text Label 9650 4250 1    50   ~ 0
+GND
+Text Label 12900 2950 1    50   ~ 0
+GND
+Text Label 2250 9250 1    50   ~ 0
+GND
+Text Label 3300 9950 1    50   ~ 0
+GND
+Text Label 3550 9950 1    50   ~ 0
+GND
+Text Label 4200 9950 1    50   ~ 0
+GND
+Text Label 5400 9950 1    50   ~ 0
+GND
+Text Label 6750 9950 1    50   ~ 0
+GND
+Text Label 8600 10000 1    50   ~ 0
+GND
+Text Label 13950 8200 1    50   ~ 0
+GND
 $EndSCHEMATC

Commit message: Tidied up 555 layout
Connections:
- net labels added: +5V_OPTO
Changed lines of the file:
@@
 Text Label 13950 8200 1    50   ~ 0
 GND
+Text Label 4250 5750 0    50   ~ 0
++5V_OPTO
 $EndSCHEMATC

Commit message: Final RevA
Parts:
- J_IN1, J_OUT1: Mfr. No: (none) -> NRJ4HF-1; Mfr: (none) -> Neutrik; MouserNo (none) -> 550-10284G; Type (none) -> Phone Connectors W/CHASSIS GROUND
- J_PWR1: Mfr. No: (none) -> RAPC722X; Mfr: (none) -> Switchcraft; MouserNo (none) -> 502-RAPC722X; Type (none) -> DC Power Connectors RT ANGL PWK JK PIN D
- P_DEPTH1: Mfr. No: (none) -> RK09L1140A5P; Mfr: (none) -> ALPS; MouserNo (none) -> 688-RK09L1140A5P; Type (none) -> 1GANG LINEAR 20% FLATTED 1TURN
- P_VOL1: Mfr. No: (none) -> RK09L1140A66; Mfr: (none) -> ALPS; MouserNo (none) -> 688-RK09L1140A66; Type (none) -> 1GANG LINEAR 20% FLATTED 1TURN
- U_BUF1: Mfr. No: (none) -> TL072SG-13; Mfr: (none) -> Diodes Incorporated; MouserNo (none) -> 621-TL072SG-13; Type (none) -> JFET INPUT OP AMP LOW NOISE
- U_INV1: Mfr. No: (none) -> TC7660SEOA713; Mfr: (none) -> Microchip Technology; MouserNo (none) -> 579-TC7660SEOA713; Type (none) -> Switching Voltage Regulators High Voltage
- U_NREG1: Mfr. No: (none) -> LM337IMP/NOPB; Mfr: (none) -> Texas Instruments; MouserNo (none) -> 926-LM337IMP/NOPB; Type (none) -> Linear Voltage Regulators 3-TERMINAL ADJ NEG REG
- U_PREG1: Mfr. No: (none) -> LM317DCYR; Mfr: (none) -> Texas Instruments; MouserNo (none) -> 595-LM317DCYR; Type (none) -> Linear Voltage Regulators 3 Term Adj. Pos.
Changed lines of the file:
@@
 F 2 "Package_SO:SOIC-8_3.9x4.9mm_P1.27mm" H 4300 8700 50  0001 C CNN
 F 3 "http://ww1.microchip.com/downloads/en/DeviceDoc/21469a.pdf" H 4300 8700 50  0001 C CNN
+F 4 "579-TC7660SEOA713" H 4200 8800 50  0001 C CNN "MouserNo"
+F 5 "TC7660SEOA713" H 4200 8800 50  0001 C CNN "Mfr. No:"
+F 6 "Microchip Technology" H 4200 8800 50  0001 C CNN "Mfr:"
+F 7 "Switching Voltage Regulators High Voltage" H 4200 8800 50  0001 C CNN "Type"
 	1    4200 8800
 	1    0    0    -1
@@
 F 2 "Package_TO_SOT_SMD:SOT-223-3_TabPin2" H 6750 8950 50  0001 C CIN
 F 3 "http://www.ti.com/lit/ds/symlink/lm317.pdf" H 6750 8700 50  0001 C CNN
+F 4 "595-LM317DCYR" H 6750 8700 50  0001 C CNN "MouserNo"
+F 5 "LM317DCYR" H 6750 8700 50  0001 C CNN "Mfr. No:"
+F 6 "Texas Instruments" H 6750 8700 50  0001 C CNN "Mfr:"
+F 7 "Linear Voltage Regulators 3 Term Adj. Pos." H 6750 8700 50  0001 C CNN "Type"
 	1    6750 8700
 	1    0    0    -1
@@
 F 2 "Package_SO:SOIC-8_3.9x4.9mm_P1.27mm" H 5700 2200 50  0001 C CNN
 F 3 "http://www.ti.com/lit/ds/symlink/tl071.pdf" H 5700 2200 50  0001 C CNN
+F 4 "621-TL072SG-13" H 5700 2200 50  0001 C CNN "MouserNo"
+F 5 "TL072SG-13" H 5700 2200 50  0001 C CNN "Mfr. No:"
+F 6 "Diodes Incorporated" H 5700 2200 50  0001 C CNN "Mfr:"
+F 7 "JFET INPUT OP AMP LOW NOISE" H 5700 2200 50  0001 C CNN "Type"
 	1    5700 2200
 	1    0    0    -1
@@
 F 2 "Potentiometer_THT:Potentiometer_Alps_RK09L_Single_Vertical" H 7550 2450 50  0001 C CNN
 F 3 "https://www.mouser.co.uk/datasheet/2/15/RK09L-1370814.pdf" H 7550 2450 50  0001 C CNN
+F 4 "688-RK09L1140A5P" H 7550 2450 50  0001 C CNN "MouserNo"
+F 5 "RK09L1140A5P" H 7550 2450 50  0001 C CNN "Mfr. No:"
+F 6 "ALPS" H 7550 2450 50  0001 C CNN "Mfr:"
+F 7 "1GANG LINEAR 20% FLATTED 1TURN" H 7550 2450 50  0001 C CNN "Type"
 	1    7550 2450
 	1    0    0    -1
@@
 F 2 "Potentiometer_THT:Potentiometer_Alps_RK09L_Single_Vertical" H 10150 3100 50  0001 C CNN
 F 3 "https://www.mouser.co.uk/datasheet/2/15/RK09L-1370814.pdf" H 10150 3100 50  0001 C CNN
+F 4 "688-RK09L1140A66" H 10150 3100 50  0001 C CNN "MouserNo"
+F 5 "RK09L1140A66" H 10150 3100 50  0001 C CNN "Mfr. No:"
+F 6 "ALPS" H 10150 3100 50  0001 C CNN "Mfr:"
+F 7 "1GANG LINEAR 20% FLATTED 1TURN" H 10150 3100 50  0001 C CNN "Type"
 	1    10150 3100
 	0    -1   -1   0
@@
 F 2 "Package_SO:SOIC-8_3.9x4.9mm_P1.27mm" H 10150 2300 50  0001 C CNN
 F 3 "http://www.ti.com/lit/ds/symlink/tl071.pdf" H 10150 2300 50  0001 C CNN
+F 4 "621-TL072SG-13" H 10150 2300 50  0001 C CNN "MouserNo"
+F 5 "TL072SG-13" H 10150 2300 50  0001 C CNN "Mfr. No:"
+F 6 "Diodes Incorporated" H 10150 2300 50  0001 C CNN "Mfr:"
+F 7 "JFET INPUT OP AMP LOW NOISE" H 10150 2300 50  0001 C CNN "Type"
 	2    10150 2300
 	1    0    0    -1
@@
 F 1 "Jack-DC" H 1605 9182 50  0000 C CNN
 F 2 "Connector_BarrelJack:BarrelJack_Horizontal" H 1600 8910 50  0001 C CNN
-F 3 "~" H 1600 8910 50  0001 C CNN
+F 3 "https://www.mouser.co.uk/datasheet/2/393/rapc722x_cd-371352.pdf" H 1600 8910 50  0001 C CNN
+F 4 "502-RAPC722X" H 1550 8950 50  0001 C CNN "MouserNo"
+F 5 "RAPC722X" H 1550 8950 50  0001 C CNN "Mfr. No:"
+F 6 "Switchcraft" H 1550 8950 50  0001 C CNN "Mfr:"
+F 7 "DC Power Connectors RT ANGL PWK JK PIN D" H 1550 8950 50  0001 C CNN "Type"
 	1    1550 8950
 	1    0    0    -1
@@
 F 2 "Package_TO_SOT_SMD:SOT-223-3_TabPin2" H 8600 8500 50  0001 C CIN
 F 3 "http://www.ti.com/lit/ds/symlink/lm337-n.pdf" H 8600 8700 50  0001 C CNN
+F 4 "926-LM337IMP/NOPB" H 8600 8700 50  0001 C CNN "MouserNo"
+F 5 "LM337IMP/NOPB" H 8600 8700 50  0001 C CNN "Mfr. No:"
+F 6 "Texas Instruments" H 8600 8700 50  0001 C CNN "Mfr:"
+F 7 "Linear Voltage Regulators 3-TERMINAL ADJ NEG REG" H 8600 8700 50  0001 C CNN "Type"
 	1    8600 8700
 	1    0    0    1
@@
 F 1 "JACK__MONO_2P_NC" H 13173 2400 50  0001 R CNN
 F 2 "custom_sockets:6_35MM_JACK_MONO_FlatTop" H 13650 2300 50  0001 C CNN
-F 3 "file:///Users/GB080220/Downloads/Drawing+NRJ4HF.pdf" H 13650 2300 50  0001 C CNN
+F 3 "http://www.neutrik.us/en-us/plugs-jacks/slim-jacks/nrj4hf-1" H 13650 2300 50  0001 C CNN
+F 4 "550-10284G" H 13650 2300 50  0001 C CNN "MouserNo"
+F 5 "NRJ4HF-1" H 13650 2300 50  0001 C CNN "Mfr. No:"
+F 6 "Neutrik" H 13650 2300 50  0001 C CNN "Mfr:"
+F 7 "Phone Connectors W/CHASSIS GROUND" H 13650 2300 50  0001 C CNN "Type"
 	1    13650 2300
 	-1   0    0    1
@@
 F 1 "JACK__MONO_2P_NC" H 1723 2200 50  0001 R CNN
 F 2 "custom_sockets:6_35MM_JACK_MONO_FlatTop" H 2200 2100 50  0001 C CNN
-F 3 "" H 2200 2100 50  0001 C CNN
+F 3 "http://www.neutrik.us/en-us/plugs-jacks/slim-jacks/nrj4hf-1" H 2200 2100 50  0001 C CNN
+F 4 "550-10284G" H 2200 2100 50  0001 C CNN "MouserNo"
+F 5 "NRJ4HF-1" H 2200 2100 50  0001 C CNN "Mfr. No:"
+F 6 "Neutrik" H 2200 2100 50  0001 C CNN "Mfr:"
+F 7 "Phone Connectors W/CHASSIS GROUND" H 2200 2100 50  0001 C CNN "Type"
 	1    2200 2100
 	1    0    0    1

Commit message: Final RevA
Other:
- note added: "3PDT"
- note added: "CLOCK"
- note removed: "BYPASS"
- moved on the sheet: U_BUF1C
Changed lines of the file:
@@
 L Amplifier_Operational:TL072 U_BUF1
 U 3 1 5BE1E2F5
-P 14700 8000
-F 0 "U_BUF1" H 14657 8045 50  0000 L CNN
-F 1 "TL072" H 14657 7956 50  0000 L CNN
-F 2 "Package_SO:SOIC-8_3.9x4.9mm_P1.27mm" H 14700 8000 50  0001 C CNN
-F 3 "http://www.ti.com/lit/ds/symlink/tl071.pdf" H 14700 8000 50  0001 C CNN
-	3    14700 8000
-	1    0    0    -1
-$EndComp
-Wire Wire Line
-	14600 7700 14600 7600
+P 10900 8900
+F 0 "U_BUF1" H 10857 8945 50  0000 L CNN
+F 1 "TL072" H 10857 8856 50  0000 L CNN
+F 2 "Package_SO:SOIC-8_3.9x4.9mm_P1.27mm" H 10900 8900 50  0001 C CNN
+F 3 "http://www.ti.com/lit/ds/symlink/tl071.pdf" H 10900 8900 50  0001 C CNN
+	3    10900 8900
+	1    0    0    -1
+$EndComp
+Wire Wire Line
+	10800 8600 10800 8500
 $Comp
 L power:+5V #PWR015
 U 1 1 5BE1F4DB
-P 14600 6950
-F 0 "#PWR015" H 14600 6800 50  0001 C CNN
-F 1 "+5V" H 14615 7121 50  0000 C CNN
-F 2 "" H 14600 6950 50  0001 C CNN
-F 3 "" H 14600 6950 50  0001 C CNN
-	1    14600 6950
+P 10800 7850
+F 0 "#PWR015" H 10800 7700 50  0001 C CNN
+F 1 "+5V" H 10815 8021 50  0000 C CNN
+F 2 "" H 10800 7850 50  0001 C CNN
+F 3 "" H 10800 7850 50  0001 C CNN
+	1    10800 7850
 	1    0    0    -1
 $EndComp
@@
 L power:-5V #PWR016
 U 1 1 5BE1F510
-P 14600 8950
-F 0 "#PWR016" H 14600 9050 50  0001 C CNN
-F 1 "-5V" H 14615 9121 50  0000 C CNN
-F 2 "" H 14600 8950 50  0001 C CNN
-F 3 "" H 14600 8950 50  0001 C CNN
-	1    14600 8950
+P 10800 9850
+F 0 "#PWR016" H 10800 9950 50  0001 C CNN
+F 1 "-5V" H 10815 10021 50  0000 C CNN
+F 2 "" H 10800 9850 50  0001 C CNN
+F 3 "" H 10800 9850 50  0001 C CNN
+	1    10800 9850
 	-1   0    0    1
 $EndComp
 Wire Wire Line
-	14600 8950 14600 8400
+	10800 9850 10800 9300
 $Comp
 L Device:R_POT P_DEPTH1
@@
 L Device:C C_BP3
 U 1 1 5BED3C35
-P 14150 7800
-F 0 "C_BP3" H 14100 7550 50  0000 R CNN
-F 1 "100nF" H 14100 7650 50  0000 R CNN
-F 2 "Capacitor_SMD:C_0805_2012Metric_Pad1.15x1.40mm_HandSolder" H 14188 7650 50  0001 C CNN
-F 3 "~" H 14150 7800 50  0001 C CNN
-	1    14150 7800
+P 10350 8700
+F 0 "C_BP3" H 10300 8450 50  0000 R CNN
+F 1 "100nF" H 10300 8550 50  0000 R CNN
+F 2 "Capacitor_SMD:C_0805_2012Metric_Pad1.15x1.40mm_HandSolder" H 10388 8550 50  0001 C CNN
+F 3 "~" H 10350 8700 50  0001 C CNN
+	1    10350 8700
 	1    0    0    1
 $EndComp
 Wire Wire Line
-	14150 7650 14150 7600
-Wire Wire Line
-	14150 7600 14600 7600
+	10350 8550 10350 8500
+Wire Wire Line
+	10350 8500 10800 8500
 $Comp
 L Device:C C_BP4
 U 1 1 5BED3C3D
-P 14150 8200
-F 0 "C_BP4" H 14100 8450 50  0000 R CNN
-F 1 "100nF" H 14100 8350 50  0000 R CNN
-F 2 "Capacitor_SMD:C_0805_2012Metric_Pad1.15x1.40mm_HandSolder" H 14188 8050 50  0001 C CNN
-F 3 "~" H 14150 8200 50  0001 C CNN
-	1    14150 8200
+P 10350 9100
+F 0 "C_BP4" H 10300 9350 50  0000 R CNN
+F 1 "100nF" H 10300 9250 50  0000 R CNN
+F 2 "Capacitor_SMD:C_0805_2012Metric_Pad1.15x1.40mm_HandSolder" H 10388 8950 50  0001 C CNN
+F 3 "~" H 10350 9100 50  0001 C CNN
+	1    10350 9100
 	1    0    0    1
 $EndComp
 Wire Wire Line
-	14150 8350 14150 8400
-Wire Wire Line
-	14150 8400 14600 8400
-Wire Wire Line
-	14150 8050 14150 8000
-Wire Wire Line
-	14150 8000 13950 8000
-Wire Wire Line
-	13950 8000 13950 8200
-Connection ~ 14150 8000
-Wire Wire Line
-	14150 8000 14150 7950
-Connection ~ 14600 7600
-Wire Wire Line
-	14600 7600 14600 6950
-Connection ~ 14600 8400
-Wire Wire Line
-	14600 8400 14600 8300
+	10350 9250 10350 9300
+Wire Wire Line
+	10350 9300 10800 9300
+Wire Wire Line
+	10350 8950 10350 8900
+Wire Wire Line
+	10350 8900 10150 8900
+Wire Wire Line
+	10150 8900 10150 9100
+Connection ~ 10350 8900
+Wire Wire Line
+	10350 8900 10350 8850
+Connection ~ 10800 8500
+Wire Wire Line
+	10800 8500 10800 7850
+Connection ~ 10800 9300
+Wire Wire Line
+	10800 9300 10800 9200
 $Comp
 L Device:C C_BP5
@@
 	7550 4800 7550 2600
 Wire Notes Line
-	850  7050 10000 7050
-Wire Notes Line
-	10000 7050 10000 10700
-Wire Notes Line
-	10000 10700 850  10700
-Wire Notes Line
 	850  10700 850  7050
-Wire Notes Line
-	10400 6600 15300 6600
-Wire Notes Line
-	15300 6600 15300 9400
-Wire Notes Line
-	15300 9400 10400 9400
-Wire Notes Line
-	10400 9400 10400 6600
-Text Notes 10500 6550 0    50   ~ 0
-BYPASS
-Text Notes 900  6950 0    50   ~ 0
+Text Notes 900  6950 0    146  ~ 0
 POWER SUPPLY
 Wire Wire Line
@@
 	3650 8650 3300 8650
 Wire Wire Line
-	3700 5750 4850 5750
+	3550 5750 4850 5750
 Wire Wire Line
 	7650 5100 7050 5100
@@
 L power:+5V #PWR0101
 U 1 1 5BEAD637
-P 3700 5400
-F 0 "#PWR0101" H 3700 5250 50  0001 C CNN
-F 1 "+5V" H 3715 5571 50  0000 C CNN
-F 2 "" H 3700 5400 50  0001 C CNN
-F 3 "" H 3700 5400 50  0001 C CNN
-	1    3700 5400
+P 3550 5400
+F 0 "#PWR0101" H 3550 5250 50  0001 C CNN
+F 1 "+5V" H 3565 5571 50  0000 C CNN
+F 2 "" H 3550 5400 50  0001 C CNN
+F 3 "" H 3550 5400 50  0001 C CNN
+	1    3550 5400
 	1    0    0    -1
 $EndComp
@@
 	7400 8100 7400 8700
 Wire Wire Line
-	3700 5400 3700 5750
+	3550 5400 3550 5750
 Text Label 3100 2750 1    50   ~ 0
 GND
@@
 Text Label 8600 10000 1    50   ~ 0
 GND
-Text Label 13950 8200 1    50   ~ 0
+Text Label 10150 9100 1    50   ~ 0
 GND
 Text Label 4250 5750 0    50   ~ 0
 +5V_OPTO
+Text Notes 4850 3800 0    146  ~ 0
+3PDT
+Text Notes 7650 4550 0    146  ~ 0
+CLOCK
+Wire Notes Line
+	11500 10700 11500 7050
+Wire Notes Line
+	850  7050 11500 7050
+Wire Notes Line
+	850  10700 11500 10700
 $EndSCHEMATC

Commit message: Added second 555 IC bypass cap
Parts:
- R_GAIN1: value 3K9 -> 2K7
Changed lines of the file:
@@
 P 9650 3750
 F 0 "R_GAIN1" H 9720 3795 50  0000 L CNN
-F 1 "3K9" H 9720 3706 50  0000 L CNN
+F 1 "2K7" H 9720 3706 50  0000 L CNN
 F 2 "Resistor_SMD:R_0805_2012Metric_Pad1.15x1.40mm_HandSolder" V 9580 3750 50  0001 C CNN
 F 3 "~" H 9650 3750 50  0001 C CNN

Commit message: Corrected DC Jack polarity
Changed lines of the file:
@@
 F 7 "DC Power Connectors RT ANGL PWK JK PIN D" H 1550 8950 50  0001 C CNN "Type"
 	1    1550 8950
-	1    0    0    -1
+	1    0    0    1
 $EndComp
 Wire Wire Line
