File: Atomizer/hardware/_autosave-Atomizer.kicad_pcb (KiCad board)
At the start: 2 copper layers, 54.6 x 98.6 mm, 49 parts

Commit message: Finished Atomizer RevB
Changed lines of the file:
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@@
     (descr "Potentiometer, vertical, Alps RK09L Single, http://www.alps.com/prod/info/E/HTML/Potentiometer/RotaryPotentiometers/RK09L/RK09L_list.html")
     (tags "Potentiometer vertical Alps RK09L Single")
-    (fp_text reference P_OSCON1 (at 5.725 -10.5 90) (layer F.SilkS)
+    (fp_text reference P_OSCON1 (at -1.905 -2.54 180) (layer F.SilkS)
       (effects (font (size 0.5 0.5) (thickness 0.125)))
     )
@@
   (segment (start 61.985 95.885) (end 61.985 93.98) (width 0.5) (layer F.Cu) (net 2))
   (segment (start 54.61 83.566) (end 54.61 77.47) (width 0.75) (layer F.Cu) (net 2))
-  (segment (start 56.896 79.62) (end 56.896 77.342) (width 0.5) (layer F.Cu) (net 2))
+  (segment (start 56.896 79.62) (end 56.896 77.342) (width 0.75) (layer F.Cu) (net 2))
   (segment (start 54.738 77.342) (end 54.61 77.47) (width 0.5) (layer F.Cu) (net 2))
-  (segment (start 56.896 77.342) (end 54.738 77.342) (width 0.5) (layer F.Cu) (net 2))
+  (segment (start 56.896 77.342) (end 54.738 77.342) (width 0.75) (layer F.Cu) (net 2))
   (via (at 87.249 137.795) (size 0.8) (drill 0.4) (layers F.Cu B.Cu) (net 3))
   (via (at 87.249 139.065) (size 0.8) (drill 0.4) (layers F.Cu B.Cu) (net 3))
