File: Atomizer/hardware/Atomizer_3PDT.sch (KiCad schematic (older format))
At the start: 3 parts

Commit message: Updated BOM. Converted to Mouser list. Moved LED away from switch
Parts:
- J_AUXTOMAIN1, J_MAINTOAUX1: MouserNo (none) -> 538-22-28-4102
Changed lines of the file:
@@
 F 2 "CustomHeaders:IDCHeader_02x05_P2.54mm_Vertical_Clockwise" H 3600 3400 50  0001 C CNN
 F 3 "~" H 3600 3400 50  0001 C CNN
+F 4 "538-22-28-4102" H 3600 3400 50  0001 C CNN "MouserNo"
 	1    3600 3400
 	1    0    0    -1
@@
 F 2 "CustomHeaders:IDCHeader_02x05_P2.54mm_Vertical_Counter_Clockwise" H 5400 3400 50  0001 C CNN
 F 3 "~" H 5400 3400 50  0001 C CNN
+F 4 "538-22-28-4102" H 5400 3400 50  0001 C CNN "MouserNo"
 	1    5400 3400
 	1    0    0    -1
