File: Atomizer/hardware/Atomizer_Clock.sch (KiCad schematic (older format))
At the start: 18 parts

Commit message: Added Atomizer Design and Code
Parts:
- added D_LED_ACT_HI1, D_LED_ACT_LO1: LED, LED_THT:LED_D5.0mm, symbol Device:LED
- added D_LED_ACT_HI2, D_LED_ACT_HI3, D_LED_ACT_LO2, D_LED_ACT_LO3: 1N914_VF1, Diode_SMD:D_SOD-123, symbol Device:D
- added R_MODE_LED1: 22K, Resistor_SMD:R_0805_2012Metric_Pad1.15x1.40mm_HandSolder, symbol Device:R
- added R_MODE_LED_PD1: 47K, Resistor_SMD:R_0805_2012Metric_Pad1.15x1.40mm_HandSolder, symbol Device:R
- R_LPF1: value 100R -> 10K
- R_MODE1: footprint (none) -> Resistor_SMD:R_0805_2012Metric_Pad1.15x1.40mm_HandSolder
- SW_MODE1: footprint (none) -> Button_Switch_THT:SW_TH_Tactile_Omron_B3F-10xx
Connections:
- net labels added: CLK_OUT_PIN, FREQ_ADJ_OFF_PIN, FREQ_ADJ_ON_PIN, MODE_BTN_PIN, MODE_LED_PIN
- net labels removed: CLKOUT, FREQ_ADJ_OFF, FREQ_ADJ_ON, MODEBTN
- wire segments 49 -> 67
- no-connect marks 2 -> 1
Other:
- note added: "Diodes prevent switch on when \nMODE_LED_PIN is in Tri-State"
- moved on the sheet: P_OSCOFF1, P_OSCON1, R_MODE1, R_OSCOFF1, R_OSCON1

Commit message: Added 3d Model
Parts:
- D_LED_ACT_HI1, D_LED_ACT_LO1: footprint LED_THT:LED_D5.0mm -> LED_THT:LED_D3.0mm
- R_LPF1: value 10K -> 100R
- SW_MODE1: footprint Button_Switch_THT:SW_TH_Tactile_Omron_B3F-10xx -> TE_Alcoswitch_Tactile_FSM_RAJ:SW_TH_Tactile_Omron_B3F-10xx
- U_OPTO1: value LTV-357T -> ACPL-217
Other:
- note added: "(ICSP Debug \nUse Only)"
Changed lines of the file:
@@
 P 6000 2700
 F 0 "R_LPF1" V 5750 2700 50  0000 C CNN
-F 1 "10K" V 5850 2700 50  0000 C CNN
+F 1 "100R" V 5850 2700 50  0000 C CNN
 F 2 "Resistor_SMD:R_0805_2012Metric_Pad1.15x1.40mm_HandSolder" V 5930 2700 50  0001 C CNN
 F 3 "~" H 6000 2700 50  0001 C CNN
@@
 P 8700 2100
 F 0 "U_OPTO1" V 8750 2650 50  0000 R CNN
-F 1 "LTV-357T" V 8650 2650 50  0000 R CNN
+F 1 "ACPL-217" V 8650 2650 50  0000 R CNN
 F 2 "Package_SO:SO-4_4.4x2.3mm_P1.27mm" H 8500 1900 50  0001 L CIN
-F 3 "https://docs.broadcom.com/docs/av02-0470en" H 8700 2100 50  0001 L CNN
+F 3 "https://docs-emea.rs-online.com/webdocs/163c/0900766b8163ccc8.pdf" H 8700 2100 50  0001 L CNN
 F 4 "630-ACPL-217-50BE" H 8700 2100 50  0001 C CNN "MouserNo"
 F 5 "ACPL-217-50BE" H 8700 2100 50  0001 C CNN "Mfr. No:"
@@
 F 0 "SW_MODE1" V 4255 6647 50  0000 L CNN
 F 1 "SW_SPST" V 4344 6647 50  0000 L CNN
-F 2 "Button_Switch_THT:SW_TH_Tactile_Omron_B3F-10xx" H 4300 6550 50  0001 C CNN
+F 2 "TE_Alcoswitch_Tactile_FSM_RAJ:SW_TH_Tactile_Omron_B3F-10xx" H 4300 6550 50  0001 C CNN
 F 3 "" H 4300 6550 50  0001 C CNN
 	1    4300 6550
@@
 F 0 "D_LED_ACT_LO1" H 6750 5100 50  0000 C CNN
 F 1 "LED" H 6750 5200 50  0000 C CNN
-F 2 "LED_THT:LED_D5.0mm" H 6750 5350 50  0001 C CNN
+F 2 "LED_THT:LED_D3.0mm" H 6750 5350 50  0001 C CNN
 F 3 "~" H 6750 5350 50  0001 C CNN
 	1    6750 5350
@@
 F 0 "D_LED_ACT_HI1" H 6750 5600 50  0000 C CNN
 F 1 "LED" H 6750 5500 50  0000 C CNN
-F 2 "LED_THT:LED_D5.0mm" H 6750 5750 50  0001 C CNN
+F 2 "LED_THT:LED_D3.0mm" H 6750 5750 50  0001 C CNN
 F 3 "~" H 6750 5750 50  0001 C CNN
 	1    6750 5750
@@
 	-1   0    0    1
 $EndComp
+Text Notes 5100 6025 0    50   ~ 0
+(ICSP Debug \nUse Only)
 $EndSCHEMATC

Commit message: Finished Atomizer RevB
Parts:
- removed C_LPFOPT1: 100nF, Capacitor_SMD:C_0805_2012Metric_Pad1.15x1.40mm_HandSolder, symbol Device:C
- removed C_LPFOPT2: 10uF, Capacitor_SMD:C_0805_2012Metric_Pad1.15x1.40mm_HandSolder, symbol Device:C
- removed R_MODE_LED_PD1: 47K, Resistor_SMD:R_0805_2012Metric_Pad1.15x1.40mm_HandSolder, symbol Device:R
- removed R_OSCLIMIT1: 330R, Resistor_SMD:R_0805_2012Metric_Pad1.15x1.40mm_HandSolder, symbol Device:R
- added J_ICSP1: Conn_02x03_Odd_Even, Connector_PinHeader_2.54mm:PinHeader_2x03_P2.54mm_Vertical, symbol Connector_Generic:Conn_02x03_Odd_Even
Connections:
- net labels added: RESET
- wire segments 67 -> 73
- no-connect marks 1 -> 0
Other:
- note added: "GND"
- note added: "MISO"
- note added: "MOSI"
- note added: "RESET"
- note added: "SCK"
- note added: "VCC"
- note removed: "(ICSP Debug \nUse Only)"
- note removed: "(Optional)"
- moved on the sheet: CP_FAST1, CP_SLOW1, C_BP1, C_BP2, D_LED1, D_LED_ACT_HI1, D_LED_ACT_HI2, D_LED_ACT_HI3, D_LED_ACT_LO1, D_LED_ACT_LO2, D_LED_ACT_LO3, P_OSCOFF1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

Commit message: Finished Atomizer RevB
Parts:
- added D_LED_ACT_HI4, D_LED_ACT_LO4: 1N914_VF1, Diode_SMD:D_SOD-123, symbol Device:D
- R_LPF1: value 100R -> 1K
Connections:
- wire segments 73 -> 75
Changed lines of the file:
@@
 P 6000 2600
 F 0 "R_LPF1" V 5750 2600 50  0000 C CNN
-F 1 "100R" V 5850 2600 50  0000 C CNN
+F 1 "1K" V 5850 2600 50  0000 C CNN
 F 2 "Resistor_SMD:R_0805_2012Metric_Pad1.15x1.40mm_HandSolder" V 5930 2600 50  0001 C CNN
 F 3 "~" H 6000 2600 50  0001 C CNN
@@
 	8125 5025 8625 5025
 Wire Wire Line
-	9925 5025 9925 4625
-Text HLabel 9925 4625 1    50   Input ~ 0
+	10575 5025 10575 4625
+Text HLabel 10575 4625 1    50   Input ~ 0
 VCC
 Wire Wire Line
 	8625 5425 8125 5425
 Wire Wire Line
-	9675 5425 9925 5425
-Wire Wire Line
-	9925 5425 9925 5825
-Text HLabel 9925 5825 3    50   Input ~ 0
+	10325 5425 10575 5425
+Wire Wire Line
+	10575 5425 10575 5825
+Text HLabel 10575 5825 3    50   Input ~ 0
 GND
 Text Notes 8575 5275 0    50   ~ 0
@@
 	4700 2700 5400 2700
 Wire Wire Line
-	9675 5025 9925 5025
+	10325 5025 10575 5025
 $Comp
 L Device:D D_LED_ACT_LO3
@@
 $EndComp
 Wire Wire Line
-	4700 2600 5850 2600
-Wire Wire Line
 	2100 2700 2900 2700
 Wire Wire Line
@@
 Wire Wire Line
 	4100 950  4100 1550
+Wire Wire Line
+	4700 2600 5850 2600
+$Comp
+L Device:D D_LED_ACT_LO4
+U 1 1 5C016653
+P 10175 5025
+F 0 "D_LED_ACT_LO4" H 10175 5275 50  0000 C CNN
+F 1 "1N914_VF1" H 10175 5149 50  0000 C CNN
+F 2 "Diode_SMD:D_SOD-123" H 10175 5025 50  0001 C CNN
+F 3 "~" H 10175 5025 50  0001 C CNN
+	1    10175 5025
+	1    0    0    -1
+$EndComp
+$Comp
+L Device:D D_LED_ACT_HI4
+U 1 1 5C0166B1
+P 10175 5425
+F 0 "D_LED_ACT_HI4" H 10175 5575 50  0000 C CNN
+F 1 "1N914_VF1" H 10175 5675 50  0000 C CNN
+F 2 "Diode_SMD:D_SOD-123" H 10175 5425 50  0001 C CNN
+F 3 "~" H 10175 5425 50  0001 C CNN
+	1    10175 5425
+	-1   0    0    1
+$EndComp
+Wire Wire Line
+	9675 5025 10025 5025
+Wire Wire Line
+	9675 5425 10025 5425
 $EndSCHEMATC

Commit message: Finished Atomizer RevA
Parts:
- removed SW_MODE1: SW_SPST, TE_Alcoswitch_Tactile_FSM_RAJ:SW_TH_Tactile_Omron_B3F-10xx, symbol Switch:SW_SPST
- added SW_MODE1: 1-1825910-4, TE_Alcoswitch_Tactile_1-1825910-4:TE_1-1825910-4, symbol TE_Alcoswitch_Tactile_1-1825910-4:1-1825910-4
- renumbered D_LED_ACT_HI2 to D_HI1, D_LED_ACT_HI3 to D_HI2, D_LED_ACT_HI4 to D_HI3, D_LED_ACT_HI1 to D_LEDHI1, D_LED_ACT_LO1 to D_LEDLO1, D_LED_ACT_LO2 to D_LO1, D_LED_ACT_LO3 to D_LO2, D_LED_ACT_LO4 to D_LO3, R_MODE_LED1 to R_MLED1
Connections:
- no-connect marks 0 -> 2
Changed lines of the file:
@@
 Text HLabel 3700 6725 3    50   Input ~ 0
 GND
-$Comp
-L Switch:SW_SPST SW_MODE1
-U 1 1 5BFD81F6
-P 5525 6225
-F 0 "SW_MODE1" V 5480 6322 50  0000 L CNN
-F 1 "SW_SPST" V 5569 6322 50  0000 L CNN
-F 2 "TE_Alcoswitch_Tactile_FSM_RAJ:SW_TH_Tactile_Omron_B3F-10xx" H 5525 6225 50  0001 C CNN
-F 3 "" H 5525 6225 50  0001 C CNN
-	1    5525 6225
-	0    1    1    0
-$EndComp
-Wire Wire Line
-	5525 6025 5525 5725
-Wire Wire Line
-	5525 6425 5525 6725
 Text HLabel 5525 6725 3    50   Input ~ 0
 GND
@@
 MODE_LED_PIN
 $Comp
-L Device:LED D_LED_ACT_LO1
+L Device:LED D_LEDLO1
 U 1 1 5BFC1538
 P 7975 5025
-F 0 "D_LED_ACT_LO1" H 7975 4775 50  0000 C CNN
+F 0 "D_LEDLO1" H 7975 4775 50  0000 C CNN
 F 1 "LED" H 7975 4875 50  0000 C CNN
 F 2 "LED_THT:LED_D3.0mm" H 7975 5025 50  0001 C CNN
@@
 $EndComp
 $Comp
-L Device:LED D_LED_ACT_HI1
+L Device:LED D_LEDHI1
 U 1 1 5BFC1588
 P 7975 5425
-F 0 "D_LED_ACT_HI1" H 7975 5275 50  0000 C CNN
+F 0 "D_LEDHI1" H 7975 5275 50  0000 C CNN
 F 1 "LED" H 7975 5175 50  0000 C CNN
 F 2 "LED_THT:LED_D3.0mm" H 7975 5425 50  0001 C CNN
@@
 $EndComp
 $Comp
-L Device:R R_MODE_LED1
+L Device:R R_MLED1
 U 1 1 5BFC269C
 P 7275 5225
-F 0 "R_MODE_LED1" V 7071 5225 50  0000 C CNN
+F 0 "R_MLED1" V 7071 5225 50  0000 C CNN
 F 1 "22K" V 7160 5225 50  0000 C CNN
 F 2 "Resistor_SMD:R_0805_2012Metric_Pad1.15x1.40mm_HandSolder" V 7205 5225 50  0001 C CNN
@@
 	10325 5025 10575 5025
 $Comp
-L Device:D D_LED_ACT_LO3
+L Device:D D_LO2
 U 1 1 5BFC855E
 P 9525 5025
-F 0 "D_LED_ACT_LO3" H 9525 5275 50  0000 C CNN
+F 0 "D_LO2" H 9525 5275 50  0000 C CNN
 F 1 "1N914_VF1" H 9525 5149 50  0000 C CNN
 F 2 "Diode_SMD:D_SOD-123" H 9525 5025 50  0001 C CNN
@@
 	8925 5025 9375 5025
 $Comp
-L Device:D D_LED_ACT_LO2
+L Device:D D_LO1
 U 1 1 5BFC8500
 P 8775 5025
-F 0 "D_LED_ACT_LO2" H 8775 5275 50  0000 C CNN
+F 0 "D_LO1" H 8775 5275 50  0000 C CNN
 F 1 "1N914_VF1" H 8775 5149 50  0000 C CNN
 F 2 "Diode_SMD:D_SOD-123" H 8775 5025 50  0001 C CNN
@@
 	9375 5425 8925 5425
 $Comp
-L Device:D D_LED_ACT_HI3
+L Device:D D_HI2
 U 1 1 5BFCED00
 P 9525 5425
-F 0 "D_LED_ACT_HI3" H 9525 5575 50  0000 C CNN
+F 0 "D_HI2" H 9525 5575 50  0000 C CNN
 F 1 "1N914_VF1" H 9525 5675 50  0000 C CNN
 F 2 "Diode_SMD:D_SOD-123" H 9525 5425 50  0001 C CNN
@@
 $EndComp
 $Comp
-L Device:D D_LED_ACT_HI2
+L Device:D D_HI1
 U 1 1 5BFCED06
 P 8775 5425
-F 0 "D_LED_ACT_HI2" H 8775 5575 50  0000 C CNN
+F 0 "D_HI1" H 8775 5575 50  0000 C CNN
 F 1 "1N914_VF1" H 8775 5675 50  0000 C CNN
 F 2 "Diode_SMD:D_SOD-123" H 8775 5425 50  0001 C CNN
@@
 	4700 2600 5850 2600
 $Comp
-L Device:D D_LED_ACT_LO4
+L Device:D D_LO3
 U 1 1 5C016653
 P 10175 5025
-F 0 "D_LED_ACT_LO4" H 10175 5275 50  0000 C CNN
+F 0 "D_LO3" H 10175 5275 50  0000 C CNN
 F 1 "1N914_VF1" H 10175 5149 50  0000 C CNN
 F 2 "Diode_SMD:D_SOD-123" H 10175 5025 50  0001 C CNN
@@
 $EndComp
 $Comp
-L Device:D D_LED_ACT_HI4
+L Device:D D_HI3
 U 1 1 5C0166B1
 P 10175 5425
-F 0 "D_LED_ACT_HI4" H 10175 5575 50  0000 C CNN
+F 0 "D_HI3" H 10175 5575 50  0000 C CNN
 F 1 "1N914_VF1" H 10175 5675 50  0000 C CNN
 F 2 "Diode_SMD:D_SOD-123" H 10175 5425 50  0001 C CNN
@@
 Wire Wire Line
 	9675 5425 10025 5425
+$Comp
+L TE_Alcoswitch_Tactile_1-1825910-4:1-1825910-4 SW_MODE1
+U 1 1 5C02509D
+P 5625 6150
+F 0 "SW_MODE1" V 5629 6291 50  0000 L CNN
+F 1 "1-1825910-4" V 5720 6291 50  0000 L CNN
+F 2 "TE_Alcoswitch_Tactile_1-1825910-4:TE_1-1825910-4" H 5625 6150 50  0001 L BNN
+F 3 "C10" H 5625 6150 50  0001 L BNN
+F 4 "TE CONNECTIVITY" H 5625 6150 50  0001 L BNN "Field4"
+F 5 "MANUFACTURER RECOMMENDATION" H 5625 6150 50  0001 L BNN "Field5"
+	1    5625 6150
+	0    1    1    0
+$EndComp
+Wire Wire Line
+	5525 5725 5525 5950
+Wire Wire Line
+	5525 6450 5525 6725
+NoConn ~ 5725 5950
+NoConn ~ 5725 6450
 $EndSCHEMATC

Commit message: Updated BOM
Parts:
- SW_MODE1: footprint TE_Alcoswitch_Tactile_1-1825910-4:TE_1-1825910-4 -> TE_Alcoswitch_Tactile_2-1825910-7:SW_2-1825910-7
Changed lines of the file:
@@
 F 0 "SW_MODE1" V 5629 6291 50  0000 L CNN
 F 1 "1-1825910-4" V 5720 6291 50  0000 L CNN
-F 2 "TE_Alcoswitch_Tactile_1-1825910-4:TE_1-1825910-4" H 5625 6150 50  0001 L BNN
+F 2 "TE_Alcoswitch_Tactile_2-1825910-7:SW_2-1825910-7" H 5625 6150 50  0001 L BNN
 F 3 "C10" H 5625 6150 50  0001 L BNN
 F 4 "TE CONNECTIVITY" H 5625 6150 50  0001 L BNN "Field4"

Commit message: Updated BOM. Converted to Mouser list. Moved LED away from switch
Parts:
- C_BP1: MouserNo (none) -> 710-885012207098; Package/Case (none) -> 0805
- C_BP2: MouserNo (none) -> 81-GRM21BC81C106KE5K; Package/Case (none) -> 0805
- D_HI1, D_HI2, D_LO1, D_LO2, D_LO3: MouserNo (none) -> 821-1N914BWRH; Package/Case (none) -> SOD-123
- D_HI3: MouserNo (none) -> 821-1N914BWRH
- D_LED1: MouserNo (none) -> 859-LTL-307EE
- D_LEDHI1, D_LEDLO1: MouserNo (none) -> 941-C4SMABGFCR2T3451
- J_ICSP1: MouserNo (none) -> 538-22-28-4062
- R_LPF1, R_MODE1, R_OSCOFF1, R_OSCON1: MouserNo (none) -> 279-CRGP0805F1K0; Package/Case (none) -> 0805; Type (none) -> 1%
- R_MLED1: MouserNo (none) -> 667-ERJ-6ENF2202V; Package/Case (none) -> 0805; Type (none) -> 1%
- SW_MODE1: MouserNo (none) -> 506-1-1825910-4
- U_CLK1: MouserNo (none) -> 556-ATTINY85-20SU
Changed lines of the file:
@@
 F 2 "LED_THT:LED_D5.0mm" H 6600 2600 50  0001 C CNN
 F 3 "~" H 6600 2600 50  0001 C CNN
+F 4 "859-LTL-307EE" H 6600 2600 50  0001 C CNN "MouserNo"
 	1    6600 2600
 	-1   0    0    1
@@
 F 2 "Resistor_SMD:R_0805_2012Metric_Pad1.15x1.40mm_HandSolder" V 5930 2600 50  0001 C CNN
 F 3 "~" H 6000 2600 50  0001 C CNN
+F 4 "279-CRGP0805F1K0" H 6000 2600 50  0001 C CNN "MouserNo"
+F 5 "1%" H 6000 2600 50  0001 C CNN "Type"
+F 6 "0805" H 6000 2600 50  0001 C CNN "Package/Case"
 	1    6000 2600
 	0    1    1    0
@@
 F 2 "Resistor_SMD:R_0805_2012Metric_Pad1.15x1.40mm_HandSolder" V 3630 5575 50  0001 C CNN
 F 3 "~" H 3700 5575 50  0001 C CNN
+F 4 "279-CRGP0805F1K0" H 3700 5575 50  0001 C CNN "MouserNo"
+F 5 "1%" H 3700 5575 50  0001 C CNN "Type"
+F 6 "0805" H 3700 5575 50  0001 C CNN "Package/Case"
 	1    3700 5575
 	-1   0    0    1
@@
 F 2 "Resistor_SMD:R_0805_2012Metric_Pad1.15x1.40mm_HandSolder" V 4655 5575 50  0001 C CNN
 F 3 "~" H 4725 5575 50  0001 C CNN
+F 4 "279-CRGP0805F1K0" H 4725 5575 50  0001 C CNN "MouserNo"
+F 5 "1%" H 4725 5575 50  0001 C CNN "Type"
+F 6 "0805" H 4725 5575 50  0001 C CNN "Package/Case"
 	1    4725 5575
 	-1   0    0    1
@@
 F 2 "Capacitor_SMD:C_0805_2012Metric_Pad1.15x1.40mm_HandSolder" H 4538 1575 50  0001 C CNN
 F 3 "~" H 4500 1725 50  0001 C CNN
+F 4 "710-885012207098" H 4500 1725 50  0001 C CNN "MouserNo"
+F 5 "0805" H 4500 1725 50  0001 C CNN "Package/Case"
 	1    4500 1725
 	1    0    0    -1
@@
 F 2 "Capacitor_SMD:C_0805_2012Metric_Pad1.15x1.40mm_HandSolder" H 5038 1575 50  0001 C CNN
 F 3 "~" H 5000 1725 50  0001 C CNN
+F 4 "81-GRM21BC81C106KE5K" H 5000 1725 50  0001 C CNN "MouserNo"
+F 5 "0805" H 5000 1725 50  0001 C CNN "Package/Case"
 	1    5000 1725
 	1    0    0    -1
@@
 F 2 "Package_SO:SOIJ-8_5.3x5.3mm_P1.27mm" H 4100 2800 50  0001 C CIN
 F 3 "http://ww1.microchip.com/downloads/en/DeviceDoc/atmel-2586-avr-8-bit-microcontroller-attiny25-attiny45-attiny85_datasheet.pdf" H 4100 2800 50  0001 C CNN
+F 4 "556-ATTINY85-20SU" H 4100 2800 50  0001 C CNN "MouserNo"
 	1    4100 2800
 	1    0    0    -1
@@
 F 2 "Resistor_SMD:R_0805_2012Metric_Pad1.15x1.40mm_HandSolder" V 5455 5575 50  0001 C CNN
 F 3 "~" H 5525 5575 50  0001 C CNN
+F 4 "279-CRGP0805F1K0" H 5525 5575 50  0001 C CNN "MouserNo"
+F 5 "1%" H 5525 5575 50  0001 C CNN "Type"
+F 6 "0805" H 5525 5575 50  0001 C CNN "Package/Case"
 	1    5525 5575
 	1    0    0    -1
@@
 F 2 "LED_THT:LED_D3.0mm" H 7975 5025 50  0001 C CNN
 F 3 "~" H 7975 5025 50  0001 C CNN
+F 4 "941-C4SMABGFCR2T3451" H 7975 5025 50  0001 C CNN "MouserNo"
 	1    7975 5025
 	1    0    0    1
@@
 F 2 "LED_THT:LED_D3.0mm" H 7975 5425 50  0001 C CNN
 F 3 "~" H 7975 5425 50  0001 C CNN
+F 4 "941-C4SMABGFCR2T3451" H 7975 5425 50  0001 C CNN "MouserNo"
 	1    7975 5425
 	-1   0    0    -1
@@
 F 2 "Resistor_SMD:R_0805_2012Metric_Pad1.15x1.40mm_HandSolder" V 7205 5225 50  0001 C CNN
 F 3 "~" H 7275 5225 50  0001 C CNN
+F 4 "667-ERJ-6ENF2202V" H 7275 5225 50  0001 C CNN "MouserNo"
+F 5 "1%" H 7275 5225 50  0001 C CNN "Type"
+F 6 "0805" H 7275 5225 50  0001 C CNN "Package/Case"
 	1    7275 5225
 	0    1    1    0
@@
 F 2 "Diode_SMD:D_SOD-123" H 9525 5025 50  0001 C CNN
 F 3 "~" H 9525 5025 50  0001 C CNN
+F 4 "821-1N914BWRH" H 9525 5025 50  0001 C CNN "MouserNo"
+F 5 "SOD-123" H 9525 5025 50  0001 C CNN "Package/Case"
 	1    9525 5025
 	1    0    0    -1
@@
 F 2 "Diode_SMD:D_SOD-123" H 8775 5025 50  0001 C CNN
 F 3 "~" H 8775 5025 50  0001 C CNN
+F 4 "821-1N914BWRH" H 8775 5025 50  0001 C CNN "MouserNo"
+F 5 "SOD-123" H 8775 5025 50  0001 C CNN "Package/Case"
 	1    8775 5025
 	1    0    0    -1
@@
 F 2 "Diode_SMD:D_SOD-123" H 9525 5425 50  0001 C CNN
 F 3 "~" H 9525 5425 50  0001 C CNN
+F 4 "821-1N914BWRH" H 9525 5425 50  0001 C CNN "MouserNo"
+F 5 "SOD-123" H 9525 5425 50  0001 C CNN "Package/Case"
 	1    9525 5425
 	-1   0    0    1
@@
 F 2 "Diode_SMD:D_SOD-123" H 8775 5425 50  0001 C CNN
 F 3 "~" H 8775 5425 50  0001 C CNN
+F 4 "821-1N914BWRH" H 8775 5425 50  0001 C CNN "MouserNo"
+F 5 "SOD-123" H 8775 5425 50  0001 C CNN "Package/Case"
 	1    8775 5425
 	-1   0    0    1
@@
 F 2 "Connector_PinHeader_2.54mm:PinHeader_2x03_P2.54mm_Vertical" H 1800 2700 50  0001 C CNN
 F 3 "~" H 1800 2700 50  0001 C CNN
+F 4 "538-22-28-4062" H 1800 2700 50  0001 C CNN "MouserNo"
 	1    1800 2700
 	1    0    0    -1
@@
 F 2 "Diode_SMD:D_SOD-123" H 10175 5025 50  0001 C CNN
 F 3 "~" H 10175 5025 50  0001 C CNN
+F 4 "821-1N914BWRH" H 10175 5025 50  0001 C CNN "MouserNo"
+F 5 "SOD-123" H 10175 5025 50  0001 C CNN "Package/Case"
 	1    10175 5025
 	1    0    0    -1
@@
 F 2 "Diode_SMD:D_SOD-123" H 10175 5425 50  0001 C CNN
 F 3 "~" H 10175 5425 50  0001 C CNN
+F 4 "821-1N914BWRH" H 10175 5425 50  0001 C CNN "MouserNo"
 	1    10175 5425
 	-1   0    0    1
@@
 F 2 "TE_Alcoswitch_Tactile_2-1825910-7:SW_2-1825910-7" H 5625 6150 50  0001 L BNN
 F 3 "C10" H 5625 6150 50  0001 L BNN
-F 4 "TE CONNECTIVITY" H 5625 6150 50  0001 L BNN "Field4"
-F 5 "MANUFACTURER RECOMMENDATION" H 5625 6150 50  0001 L BNN "Field5"
+F 4 "506-1-1825910-4" H 5625 6150 50  0001 C CNN "MouserNo"
+F 5 "TE CONNECTIVITY" H 5625 6150 50  0001 L BNN "Field4"
+F 6 "MANUFACTURER RECOMMENDATION" H 5625 6150 50  0001 L BNN "Field5"
 	1    5625 6150
 	0    1    1    0

Commit message: updates
Parts:
- U_CLK1: symbol MCU_Microchip_ATtiny:ATtiny85-20SU -> Atomizer-rescue:ATtiny85-20SU-MCU_Microchip_ATtiny
Changed lines of the file:
@@
 EESchema Schematic File Version 4
 LIBS:Atomizer-cache
-EELAYER 26 0
+EELAYER 29 0
 EELAYER END
 $Descr A4 11693 8268
@@
 $EndComp
 $Comp
-L MCU_Microchip_ATtiny:ATtiny85-20SU U_CLK1
+L Atomizer-rescue:ATtiny85-20SU-MCU_Microchip_ATtiny U_CLK1
 U 1 1 5BFB6DEC
 P 4100 2800
